File: summit_scourer/Kicad/summit_scourer.kicad_sch (KiCad schematic)
At the start: 3 parts, among them J2 Conn_Coaxial

Commit message: Add files via upload
Parts:
- removed C11, C12: 100n, Capacitor_SMD:C_0504_1310Metric_Pad0.83x1.28mm_HandSolder, symbol Device:C
- removed J2: Conn_Coaxial, symbol Connector:Conn_Coaxial
Other:
- added sheet RF_input_and_filtering (RF_input_and_filtering.kicad_sch)
- sheet MCU_and_UI ports: added RX_BFO, TX_LO; removed none

Commit message: Add files via upload
Parts:
- added C11, C12: 100n, Capacitor_SMD:C_0504_1310Metric_Pad0.83x1.28mm_HandSolder, symbol Device:C
- added J2: Conn_Coaxial, symbol Connector:Conn_Coaxial
Connections:
- new net: C11.2, C12.2, J2.1 (In)
- new net GND: J2.2 (Ext)
- new net RX/RF: C11.1, C12.1
Other:
- removed sheet RF_input_and_filtering
- added sheet channel_switching_and_filtering (channel_switching_and_filtering.kicad_sch)
- sheet MCU_and_UI ports: added none; removed RX_BFO, TX_LO
- sheet RX ports: added RF, RX_ant_en; removed RX_RF
