File: Kicad/summit_scourer.kicad_pcb (KiCad board)
At the start: 2 copper layers, 100 x 70 mm, 135 parts, among them J1 SI5351_breakout_board, J2 Conn_Coaxial, J3 Conn_Coaxial, J4 Audio_out, J5 Mic/Key, J6 RFShield_OnePiece, Q1 Q_NMOS, Q2 2N7002H, SW1 SW_DPDT_x3, SW2 push_btn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

Commit message: Add files via upload
Parts:
- moved U3 3.92 mm to (94.3, 72.5)
- moved C6 3.92 mm to (88.8, 76.4)
- moved C7 3.92 mm to (88.8, 74.8)
- moved L1 0.90 mm to (105.9, 60.6)
- moved Q1 0.36 mm to (103.5, 70.5)
- moved R2 0.33 mm to (108.3, 71.3)
Routing:
- net /TX/TX_PA: track 0.00 -> 18.4 mm
- net Net-(C8-Pad1): track 21.4 -> 15.3 mm
- net Net-(C47-Pad1): track 23.1 -> 18.7 mm
- net Net-(Q1-G): track 0.00 -> 4.07 mm
- net GND: track 0.00 -> 2.41 mm

Commit message: Add files via upload
Parts:
- removed J3: Conn_Coaxial, Connector_Coaxial:SMA_Amphenol_901-143_Horizontal
- added C52: 10u, Capacitor_SMD:C_1210_3225Metric_Pad1.33x2.70mm_HandSolder, F.Cu at (4.54, 44.6)
- added C53: 10u, Capacitor_SMD:C_1210_3225Metric_Pad1.33x2.70mm_HandSolder, F.Cu at (4.54, 48.8)
- added C54: 10u, Capacitor_SMD:C_1210_3225Metric_Pad1.33x2.70mm_HandSolder, F.Cu at (4.54, 53.1)
- added C55: 10u, Capacitor_SMD:C_1210_3225Metric_Pad1.33x2.70mm_HandSolder, F.Cu at (4.54, 57.3)
- added C56: 10u, Capacitor_SMD:C_1210_3225Metric_Pad1.33x2.70mm_HandSolder, F.Cu at (4.54, 61.6)
- added C57: 10u, Capacitor_SMD:C_1210_3225Metric_Pad1.33x2.70mm_HandSolder, F.Cu at (4.54, 65.8)
- added C58: 470u, Capacitor_THT:CP_Radial_D8.0mm_P3.80mm, F.Cu at (-7.56, 51.5)
- added C59: 100n, Capacitor_SMD:C_0603_1608Metric_Pad1.08x0.95mm_HandSolder, F.Cu at (-14.5, 60.1)
- added H1: Vin_+, TestPoint:TestPoint_THTPad_3.0x3.0mm_Drill1.5mm, F.Cu at (-23.3, 78.7)
- added H2: Vin_-, TestPoint:TestPoint_THTPad_3.0x3.0mm_Drill1.5mm, F.Cu at (-17.5, 79.2)
- added H3: FM_ant, TestPoint:TestPoint_THTPad_2.0x2.0mm_Drill1.0mm, F.Cu at (97.2, 100.9)
- added L9: L_Ferrite, Inductor_SMD:L_6.3x6.3_H3, F.Cu at (-6.35, 60.2)
- added R50: 0R, summit_scourer:R_0603_linked, F.Cu at (21.9, 43.7)
- added U5: AZ1117-3.3, Package_TO_SOT_SMD:TO-252-2, F.Cu at (11.8, 38.7)
- added U6: AZ1117-5.0, Package_TO_SOT_SMD:TO-252-2, F.Cu at (16.4, 54.6)
- added U7: AZ1117-3.3, Package_TO_SOT_SMD:TO-252-2, F.Cu at (14.9, 72.6)
- moved C13 9.68 mm to (90.5, 80.6)
- moved L2 9.68 mm to (73.3, 82.4)
- moved R29 9.68 mm to (73.3, 85.9)
- moved R3 9.68 mm to (65.6, 82.0)
- moved C1 9.68 mm to (85.1, 99.1)
- moved C10 9.68 mm to (92.9, 84.8)
- moved C15 9.68 mm to (80.5, 83.1)
- moved C16 9.68 mm to (92.2, 93.7)
- moved C17 9.68 mm to (64.9, 96.4)
- moved C18 9.68 mm to (82.1, 98.5)
- moved C19 9.68 mm to (75.4, 98.5)
- moved C2 9.68 mm to (87.7, 99.1)
- moved C48 9.68 mm to (67.5, 98.6)
- moved C49 9.68 mm to (73.9, 92.9)
- moved C50 9.68 mm to (79.0, 83.1)
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Connections:
- C37 pad 1: Net-(SW1B-C) -> Net-(SW1B-A)
- C38 pad 1: Net-(SW1B-C) -> Net-(SW1B-A)
- C38 pad 2: Net-(C21-Pad2) -> Net-(C38-Pad2)
- C39 pad 2: Net-(C23-Pad2) -> Net-(C39-Pad2)
- C40 pad 1: Net-(C23-Pad2) -> Net-(C39-Pad2)
- C40 pad 2: Net-(SW1C-C) -> Net-(SW1C-A)
- C41 pad 1: Net-(SW1C-C) -> Net-(SW1C-A)
- L6 pad 1: Net-(C21-Pad2) -> Net-(C38-Pad2)
- L6 pad 2: Net-(C23-Pad2) -> Net-(C39-Pad2)
- L7 pad 1: Net-(C23-Pad2) -> Net-(C39-Pad2)
- L7 pad 2: Net-(SW1C-C) -> Net-(SW1C-A)
