File: Kicad/summit_scourer.kicad_pcb (KiCad board)
At the start: 2 copper layers, 100 x 70 mm, 150 parts, among them J1 SI5351_breakout_board, J2 Conn_Coaxial, J3 PTT/Mic, J4 Internal_SPK, J5 PTT/Mic, J6 RFShield_OnePiece, Q1 Q_NMOS, Q2 2N7002H, SW1 SW_DPDT_x3, SW2 push_btn, SW3 push_btn, SW4 push_btn, SW5 push_btn, SW6 push_btn, SW7 push_btn, T1 T, T3 T, U1 SI4732-A10-GS, U2 ESP32-WROOM-32UE, U3 74AC00, U5 AZ1117-3.3, U7 AZ1117-3.3, Y1 32.768 KHz

Commit message: Add files via upload
Parts:
- removed T3: T, summit_scourer:torroid_transformer
- added C55: 10n, Capacitor_SMD:C_0603_1608Metric_Pad1.08x0.95mm_HandSolder, F.Cu at (172.8, 112.6)
- added D5: 1N4007, Diode_THT:D_A-405_P2.54mm_Vertical_AnodeUp, F.Cu at (182.4, 79.4)
- added J7: Conn_01x06_Socket, Connector_PinHeader_2.54mm:PinHeader_1x06_P2.54mm_Vertical, F.Cu at (128.3, 71.2)
- added J8: SWR_interface, Connector_PinHeader_2.54mm:PinHeader_1x05_P2.54mm_Vertical, F.Cu at (254.7, 55.7)
- added MK1: Microphone, Connector_PinHeader_2.54mm:PinHeader_1x02_P2.54mm_Vertical, F.Cu at (133.8, 106.5)
- added R34: 10k, Resistor_SMD:R_0603_1608Metric, F.Cu at (170.4, 111.7)
- added R53: 10k, Resistor_SMD:R_0603_1608Metric, F.Cu at (175.2, 111.7)
- added R54: 0R, summit_scourer:R_0603_linked, F.Cu at (167.8, 114.1)
- added T2: T, summit_scourer:torroid_transformer, F.Cu at (240.0, 56.1)
- added TP3: IO12, Connector_PinHeader_2.54mm:PinHeader_1x01_P2.54mm_Vertical, F.Cu at (120.4, 99.0)
- moved R51 119.9 mm to (126.8, 120.5), turned to 90 degrees
- moved R52 115.1 mm to (126.8, 117.3), turned to 90 degrees
- moved C30 92.5 mm to (103.6, 131.4), turned to -90 degrees
- moved C24 90.6 mm to (188.4, 115.9), turned to 180 degrees
- moved R7 90.5 mm to (106.0, 101.0), turned to -90 degrees
- moved C37 84.7 mm to (188.4, 126.9)
- moved C21 84.6 mm to (177.5, 126.8)
- moved C20 82.6 mm to (177.5, 115.9), turned to 0 degrees
- moved C52 81.4 mm to (165.1, 79.1)
- moved C59 79.8 mm to (188.1, 75.6), turned to 90 degrees
- moved C40 79.6 mm to (188.4, 125.1), turned to 0 degrees
- moved R36 78.3 mm to (133.6, 97.9)
- moved C42 78.3 mm to (132.0, 97.9)
- moved R10 77.8 mm to (100.9, 128.7)
- moved R6 77.8 mm to (100.9, 134.2)
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Connections:
- net /channel_switching_and_filtering/Forward_indicator renamed /SWR_bridge/Reverse_indicator
- net /channel_switching_and_filtering/Reverse_indicator renamed /SWR_bridge/Forward_indicator
- C11 pad 1: /RX/RF -> /TX/RF_out
- C12 pad 1: /RX/RF -> /TX/RF_out
- C14 pad 1: VBUS_filtered -> VBUS
- C20 pad 1: Net-(SW1B-C) -> Net-(SW1B-A)
- C20 pad 2: GND -> RF_GND
- C21 pad 2: Net-(C21-Pad2) -> RF_GND
- C22 pad 1: Net-(SW1C-C) -> Net-(SW1B-A)
- C22 pad 2: GND -> Net-(C22-Pad2)
- C23 pad 1: GND -> Net-(SW1B-C)
- C24 pad 1: Net-(C23-Pad2) -> RF_GND
- C24 pad 2: Net-(SW1C-C) -> Net-(C24-Pad2)
- C37 pad 1: Net-(SW1B-A) -> RF_GND
- C37 pad 2: GND -> Net-(C37-Pad2)
- C38 pad 1: Net-(SW1B-A) -> Net-(C24-Pad2)
- C38 pad 2: Net-(C38-Pad2) -> Net-(SW1C-A)
- C39 pad 1: GND -> Net-(C37-Pad2)
- C39 pad 2: Net-(C39-Pad2) -> Net-(SW1C-C)
- C40 pad 1: Net-(C39-Pad2) -> Net-(SW1C-A)
- C40 pad 2: Net-(SW1C-A) -> RF_GND
- C41 pad 1: Net-(SW1C-A) -> Net-(SW1C-C)
- C41 pad 2: GND -> RF_GND
- C53 pad 1: VBUS_filtered -> VBUS
- J2 pad 2: GND -> RF_GND
- L1 pad 1: VBUS_filtered -> VBUS
- L1 pad 2: /TX/TX_PA -> /RX/RF
- L3 pad 1: Net-(C21-Pad2) -> Net-(C22-Pad2)
- L3 pad 2: Net-(C23-Pad2) -> Net-(C24-Pad2)
- L4 pad 2: Net-(SW1C-C) -> Net-(C37-Pad2)
- L6 pad 1: Net-(C38-Pad2) -> Net-(C24-Pad2)
- L6 pad 2: Net-(C39-Pad2) -> Net-(SW1C-A)
- L7 pad 1: Net-(C39-Pad2) -> Net-(C37-Pad2)
- L7 pad 2: Net-(SW1C-A) -> Net-(SW1C-C)
- L9 pad 1: VBUS -> Net-(D5-K)
- Q1 pad 2: GND -> RF_GND
- Q1 pad 3: /TX/TX_PA -> /RX/RF
- R21 pad 1: Net-(D2-A) -> Net-(D1-A)
- R22 pad 1: Net-(D1-A) -> Net-(D2-A)
- SW1 pad 5: /TX/TX_PA -> /RX/RF
- SW1 pad 8: Net-(SW1C-B) -> /TX/RF_out
- T1 pad 1: /channel_switching_and_filtering/RF_out -> Net-(J8-Pin_2)
- T1 pad 2: Net-(SW1C-B) -> Net-(J8-Pin_1)
- U2 pad 10: /MCU_and_UI/LCD.BL -> /MCU_and_UI/TX_Mod
- U2 pad 27: unconnected-(U2-IO16-Pad27) -> /MCU_and_UI/LCD.BL
Routing:
- net Net-(SW1C-C): track 0.00 -> 38.6 mm
- net Net-(SW1C-A): track 0.00 -> 36.6 mm
- net Net-(SW1B-C): track 0.00 -> 25.7 mm, vias 0 -> 1
- net Net-(SW1B-A): track 0.00 -> 25.2 mm, vias 0 -> 1
- net Net-(C24-Pad2): track 0.00 -> 18.4 mm
- net Net-(C37-Pad2): track 0.00 -> 18.4 mm
- net /TX/TX_PA: track 18.4 -> 0.00 mm
- net /RX/RF: track 0.00 -> 18.4 mm
- net /TX/RF_out: track 0.00 -> 13.3 mm
- net +3V3: track 0.00 -> 10.4 mm
- net Net-(J2-In): track 0.00 -> 7.14 mm
- net /MCU_and_UI/LCD.D/I: track 16.0 -> 11.0 mm
- net /MCU_and_UI/LCD.R/L: track 15.7 -> 11.4 mm
- net Net-(C55-Pad1): track 0.00 -> 3.15 mm
- net Net-(Q1-G): track 4.07 -> 6.93 mm
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- added copper zone on F.Cu, net GND
- added copper zone on In1.Cu, net GND
- added copper zone on F.Cu, net Net-(D5-K)
- added copper zone on In1.Cu, net RF_GND
- added copper zone on F.Cu, net VBUS
- added copper zone on F.Cu, net VBUS_filtered
Other:
- copper layers 2 -> 4

Commit message: Add files via upload
Parts:
- removed C10, C26, C28, C43, C44, C45: 10n, Capacitor_SMD:C_0603_1608Metric_Pad1.08x0.95mm_HandSolder
- removed C19, C48, C51: 10u, Capacitor_SMD:C_1210_3225Metric_Pad1.33x2.70mm_HandSolder
- removed C27, C29, C30, C47, C50: 100n, Capacitor_SMD:C_0603_1608Metric_Pad1.08x0.95mm_HandSolder
- removed C38, C40: C, Capacitor_SMD:C_0603_1608Metric_Pad1.08x0.95mm_HandSolder
- removed D1, D2: D, Diode_SMD:D_PowerDI-123
- removed H3: FM_ant, TestPoint:TestPoint_THTPad_2.0x2.0mm_Drill1.0mm
- removed J1: SI5351_breakout_board, Connector_PinHeader_2.54mm:PinHeader_1x07_P2.54mm_Vertical
- removed J6: RFShield_OnePiece, summit_scourer:MS323_hatched
- removed L4, L7: L_Ferrite, Inductor_THT:L_Toroid_Vertical_L10.0mm_W5.0mm_P5.08mm
- removed L9: L_Ferrite, Inductor_SMD:L_6.3x6.3_H3
- removed R10, R12, R13, R14, R15, R16, R17, R20, R37: 10k, Resistor_SMD:R_0603_1608Metric
- removed R11, R36, R38, R39, R48: 0R, summit_scourer:R_0603_linked
- removed R18, R19: 1k, Resistor_SMD:R_0603_1608Metric
- removed R21, R22: 220R, Resistor_SMD:R_0603_1608Metric
- removed R23, R24, R5: 100k, Resistor_SMD:R_0603_1608Metric
- removed SW1: SW_DPDT_x3, summit_scourer:SW_GF-161-0005
- removed SW2, SW3, SW4, SW5, SW6: push_btn, Button_Switch_THT:SW_PUSH_6mm_H9.5mm
- removed T1, T2: T, summit_scourer:torroid_transformer
- removed TP3: IO12, Connector_PinHeader_2.54mm:PinHeader_1x01_P2.54mm_Vertical
- removed U2: ESP32-WROOM-32UE, RF_Module:ESP32-WROOM-32UE
- added C61: 1n, Capacitor_SMD:C_0603_1608Metric_Pad1.08x0.95mm_HandSolder, F.Cu at (180.0, 105.8)
- added C63: 100n, Capacitor_SMD:C_0603_1608Metric_Pad1.08x0.95mm_HandSolder, F.Cu at (139.3, 97.0)
- added Q3: BS170, Package_TO_SOT_THT:TO-92_Inline, F.Cu at (178.9, 81.0)
- added Q4: BS170, Package_TO_SOT_THT:TO-92_Inline, F.Cu at (184.0, 81.0)
- added RV1: 10k, Connector_PinHeader_2.54mm:PinHeader_1x03_P2.54mm_Vertical, F.Cu at (128.6, 77.2)
- added SW8: RotaryEncoder, summit_scourer:Rotary_encoder, F.Cu at (112.5, 107.0)
- added U6: LM4808MX_NOPB, Package_SO:SO-8_3.9x4.9mm_P1.27mm, F.Cu at (132.1, 91.5)
- added U8: 74AC00, Package_SO:SOIC-14_3.9x8.7mm_P1.27mm, F.Cu at (169.1, 90.8)
- added Y3: 25MHz, Crystal:Crystal_SMD_3225-4Pin_3.2x2.5mm, F.Cu at (170.0, 109.3)
- C1, C2: value 22p -> 10n
- C13, C17, C5, C8: value 10n -> 100n
- C14, C34, C42, C56, C57, C6, C9, R50, R8, U5, U7: moved to B.Cu
- C15, C32, C59: value 100n -> 10u; footprint Capacitor_SMD:C_0603_1608Metric_Pad1.08x0.95mm_HandSolder -> Capacitor_SMD:C_1210_3225Metric_Pad1.33x2.70mm_HandSolder
- C20, C21: value C -> 10n
- C22: value C -> 10n; moved to B.Cu
- C23: value C -> 10u; footprint Capacitor_SMD:C_0603_1608Metric_Pad1.08x0.95mm_HandSolder -> Capacitor_SMD:C_1210_3225Metric
- C24: value C -> 100n; moved to B.Cu
- C3: value 10u -> 22p; footprint Capacitor_SMD:C_1210_3225Metric_Pad1.33x2.70mm_HandSolder -> Capacitor_SMD:C_0603_1608Metric_Pad1.08x0.95mm_HandSolder
- C33, C36: value 100n -> 10n; moved to B.Cu
- C37, C39: value C -> 150p
- C4: value 100n -> 22p
- C41: value C -> 470p
- C46: value 10n -> 470p
- C49: value 100n -> 1n
- C52: value 10u -> 100n; footprint Capacitor_SMD:C_1210_3225Metric_Pad1.33x2.70mm_HandSolder -> Capacitor_SMD:C_0603_1608Metric_Pad1.08x0.95mm_HandSolder; moved to B.Cu
- C53: value 10u -> 150p; footprint Capacitor_SMD:C_1210_3225Metric -> Capacitor_SMD:C_0603_1608Metric_Pad1.08x0.95mm_HandSolder; moved to B.Cu
- C54: value 10u -> 470u; footprint Capacitor_SMD:C_1210_3225Metric_Pad1.33x2.70mm_HandSolder -> Capacitor_THT:CP_Radial_D8.0mm_P3.80mm
- C55: value 10n -> 150p; moved to B.Cu
- C58: value 470u -> 10u; footprint Capacitor_THT:CP_Radial_D8.0mm_P3.80mm -> Capacitor_SMD:C_1210_3225Metric_Pad1.33x2.70mm_HandSolder
- J3: moved to F.Cu
- J4: value Internal_SPK -> Headphone; footprint Connector_PinHeader_2.54mm:PinHeader_1x03_P2.54mm_Vertical -> Connector_Audio:Jack_3.5mm_CUI_SJ1-3525N_Horizontal; moved to F.Cu
- J5: value PTT/Mic -> Internal_SPK; footprint Connector_Audio:Jack_3.5mm_CUI_SJ1-3525N_Horizontal -> Connector_PinHeader_2.54mm:PinHeader_1x02_P2.54mm_Vertical; moved to F.Cu
- J7: value Conn_01x06_Socket -> Prog
- J8: value SWR_interface -> Conn_01x06_Socket; footprint Connector_PinHeader_2.54mm:PinHeader_1x05_P2.54mm_Vertical -> Connector_PinHeader_2.54mm:PinHeader_1x04_P2.54mm_Vertical
- L2: value DNF -> L_Ferrite; footprint Inductor_SMD:L_2010_5025Metric -> Inductor_SMD:L_TDK_SLF6025
- L3: value L_Ferrite -> 15T/T37-2
- L6: value L_Ferrite -> 10T/T37-2
- L8: footprint Inductor_SMD:L_TDK_SLF6025 -> Inductor_SMD:L_6.3x6.3_H3
- Q1: value Q_NMOS -> BS170; footprint Package_TO_SOT_SMD:SOT-89-3_Handsoldering -> Package_TO_SOT_THT:TO-92_Inline
- R1, R2: value 100k -> 0R; footprint Resistor_SMD:R_0603_1608Metric -> summit_scourer:R_0603_linked
- R25, R26: value 220R -> 0R; footprint Resistor_SMD:R_0603_1608Metric -> summit_scourer:R_0603_linked
- R28, R29: value 0R -> 220R; footprint summit_scourer:R_0603_linked -> Resistor_SMD:R_0603_1608Metric
- R30, R31: value 0R -> 120k; footprint summit_scourer:R_0603_linked -> Resistor_SMD:R_0603_1608Metric
- R33, R54: value 0R -> 100k; footprint summit_scourer:R_0603_linked -> Resistor_SMD:R_0603_1608Metric; moved to B.Cu
- R34, R9: value 10k -> 0R; footprint Resistor_SMD:R_0603_1608Metric -> summit_scourer:R_0603_linked; moved to B.Cu
- R35, R44, R49: value 0R -> 10k; footprint summit_scourer:R_0603_linked -> Resistor_SMD:R_0603_1608Metric
- R4: value 10k -> 0R; footprint Resistor_SMD:R_0603_1608Metric -> summit_scourer:R_0603_linked
- R40: value 0R -> 100k; footprint summit_scourer:R_0603_linked -> Resistor_SMD:R_0603_1608Metric
- R41: value 0R -> 1k; footprint summit_scourer:R_0603_linked -> Resistor_SMD:R_0603_1608Metric; moved to B.Cu
- R42, R45: value 0R -> 10k; footprint summit_scourer:R_0603_linked -> Resistor_SMD:R_0603_1608Metric; moved to B.Cu
- R46, R47, R7: value 0R -> 1k; footprint summit_scourer:R_0603_linked -> Resistor_SMD:R_0603_1608Metric
- SW7: value push_btn -> Key; footprint Button_Switch_THT:SW_PUSH_6mm_H9.5mm -> Connector_PinHeader_2.54mm:PinHeader_1x02_P2.54mm_Vertical; moved to F.Cu
- TP1: value RX_BFO -> IO12; footprint TestPoint:TestPoint_THTPad_1.5x1.5mm_Drill0.7mm -> Connector_PinHeader_2.54mm:PinHeader_1x01_P2.54mm_Vertical
- U3: value 74AC00 -> Si5351A-B-GT; footprint Package_SO:SOIC-14_3.9x8.7mm_P1.27mm -> Package_SO:MSOP-10_3x3mm_P0.5mm
- U4: value ~ -> ESP32-WROOM-32UE; footprint summit_scourer:Display_8x2 -> RF_Module:ESP32-WROOM-32UE
- moved J8 115.5 mm to (145.8, 94.2), turned to -90 degrees
- moved C46 79.7 mm to (181.2, 86.8), turned to 180 degrees
- moved R9 68.0 mm to (167.7, 104.2), turned to -90 degrees
- moved C56 59.7 mm to (148.2, 79.8), turned to 90 degrees
- moved C57 58.8 mm to (145.8, 88.0), turned to 90 degrees
- moved C18 54.2 mm to (123.3, 86.2), turned to 0 degrees
- moved L8 51.6 mm to (153.3, 85.0)
- moved C41 51.4 mm to (181.2, 85.2), turned to 180 degrees
- moved U7 51.2 mm to (137.5, 87.3)
- moved C59 50.7 mm to (138.8, 87.5)
- moved J7 49.8 mm to (111.2, 118.0)
- moved C49 49.6 mm to (180.0, 96.5), turned to 0 degrees
- moved C23 48.5 mm to (161.3, 80.0), turned to 90 degrees
- moved C21 46.5 mm to (135.5, 106.8)
- moved C39 45.4 mm to (185.3, 86.2)
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Connections:
- C1 pad 1: Net-(U1-GPO3/DCLK) -> /RX_ant_en
- C11 pad 1: /TX/RF_out -> Net-(C11-Pad1)
- C12 pad 1: /TX/RF_out -> Net-(C11-Pad1)
- C13 pad 1: Net-(Q2-S) -> Net-(U1-VDD)
- C13 pad 2: /RX/RF -> GND
- C14 pad 1: VBUS -> Net-(U8E-VCC)
- C15 pad 1: Net-(D3-K) -> Net-(U1-ROUT/DOUT)
- C15 pad 2: Net-(U1-AMI) -> Net-(C15-Pad2)
- C16 pad 1: Net-(C16-Pad1) -> Net-(U1-VDD)
- C16 pad 2: Net-(U1-FMI) -> GND
- C17 pad 1: Net-(U1-VDD) -> +3V3_RX
- C18 pad 1: Net-(U1-LOUT/DFS) -> /audio_out_right
- C18 pad 2: /MCU_and_UI/audio_out_left -> Net-(U6-OUT_A)
- C2 pad 1: Net-(U1-RCLK) -> Net-(Q2-S)
- C2 pad 2: GND -> Net-(Q1-D)
- C20 pad 1: Net-(SW1B-A) -> Net-(U8E-VCC)
- C20 pad 2: RF_GND -> GND
- C21 pad 1: Net-(SW1B-C) -> Net-(C21-Pad1)
- C21 pad 2: RF_GND -> GND
- C22 pad 1: Net-(SW1B-A) -> Net-(C22-Pad1)
- C22 pad 2: Net-(C22-Pad2) -> Net-(Q1-G)
- C23 pad 1: Net-(SW1B-C) -> VBUS
- C23 pad 2: Net-(C23-Pad2) -> GND
- C24 pad 1: RF_GND -> VBUS
- C24 pad 2: Net-(C24-Pad2) -> GND
- C25 pad 1: Net-(U2-VDD) -> /Encoder.btn
- C3 pad 1: +3V3 -> Net-(U1-RCLK)
- C31 pad 1: Net-(U4-Chip_enable) -> /ESP_reset
- C32 pad 1: /MCU_and_UI/Btn.Select -> Net-(U4-VDD)
- C33 pad 1: /MCU_and_UI/Btn.Up -> Net-(U4-VDD)
- C34 pad 1: /MCU_and_UI/Btn.Down -> /PTT_key
- C35 pad 1: /MCU_and_UI/Btn.Back -> Net-(U4-VDD)
- C36 pad 1: /MCU_and_UI/Btn.Menu -> /mic_in
- C37 pad 1: RF_GND -> Net-(Q1-D)
- C37 pad 2: Net-(C37-Pad2) -> GND
- C39 pad 1: Net-(C37-Pad2) -> Net-(Q1-D)
- C39 pad 2: Net-(SW1C-C) -> GND
- C4 pad 1: +3V3 -> Net-(U1-GPO3/DCLK)
- C41 pad 1: Net-(SW1C-C) -> Net-(Q1-D)
- C41 pad 2: RF_GND -> Net-(C41-Pad2)
- C42 pad 1: /MCU_and_UI/Band_select -> /mic_in
- C42 pad 2: GND -> Net-(C42-Pad2)
- C46 pad 1: /SWR_bridge/Forward_indicator -> Net-(Q1-D)
- C46 pad 2: GND -> Net-(C41-Pad2)
- C49 pad 1: Net-(U1-VDD) -> GND
- C49 pad 2: GND -> Net-(C49-Pad2)
- C5 pad 1: +3V3 -> Net-(D3-K)
- C5 pad 2: GND -> Net-(U1-AMI)
- C52 pad 1: +3V3 -> VBUS
- C53 pad 1: VBUS -> Net-(C49-Pad2)
- C53 pad 2: GND -> Net-(C11-Pad1)
- C55 pad 1: Net-(C55-Pad1) -> Net-(C49-Pad2)
- C55 pad 2: GND -> Net-(C11-Pad1)
- C57 pad 1: +3V3_RX -> VBUS_filtered
- C58 pad 1: VBUS_filtered -> +3V3
- C59 pad 1: VBUS -> +3V3_RX
- C6 pad 1: Net-(U3E-VCC) -> +3V3
- C7 pad 1: Net-(U3E-VCC) -> +3V3
- C8 pad 2: Net-(Q1-G) -> Net-(U3-CLK0)
- C9 pad 1: Net-(C47-Pad1) -> Net-(C8-Pad1)
- J2 pad 2: RF_GND -> GND
- J3 pad R: Net-(C30-Pad2) -> Net-(C42-Pad2)
- J3 pad RN: /MCU_and_UI/onboard_mic -> /onboard_mic
- J3 pad T: /MCU_and_UI/PTT_key -> /PTT_key
- J3 pad TN: /MCU_and_UI/onboard_key -> /onboard_key
- J7 pad 2: /MCU_and_UI/ESP_reset -> /ESP_boot
- J7 pad 4: /MCU_and_UI/ESP_RX -> /ESP_TX
- J7 pad 5: /MCU_and_UI/ESP_TX -> /ESP_reset
- J7 pad 6: /MCU_and_UI/ESP_boot -> /ESP_RX
- J8 pad 1: Net-(J8-Pin_1) -> /I2C_SDIO
- J8 pad 2: Net-(J8-Pin_2) -> /I2C_SCL
- J8 pad 3: /SWR_bridge/Forward_indicator -> +3V3
- J8 pad 4: /SWR_bridge/Reverse_indicator -> GND
- L1 pad 2: /RX/RF -> Net-(Q1-D)
- L2 pad 1: Net-(D3-K) -> Net-(U1-VDD)
- L2 pad 2: GND -> +3V3_RX
- L3 pad 1: Net-(C22-Pad2) -> Net-(C41-Pad2)
- L3 pad 2: Net-(C24-Pad2) -> Net-(C49-Pad2)
- L5 pad 1: Net-(U2-VDD) -> Net-(U4-VDD)
- L6 pad 1: Net-(C24-Pad2) -> Net-(C49-Pad2)
- L6 pad 2: Net-(SW1C-A) -> Net-(C11-Pad1)
- L8 pad 1: Net-(U1-VDD) -> Net-(D5-K)
- L8 pad 2: +3V3_RX -> VBUS_filtered
- MK1 pad 2: /MCU_and_UI/onboard_mic -> /onboard_mic
- Q1 pad 1: Net-(Q1-G) -> Net-(Q1-D)
- Q1 pad 2: RF_GND -> Net-(Q1-G)
- Q1 pad 3: /RX/RF -> GND
- Q2 pad 1: Net-(Q2-G) -> /RX_ant_en
- R1 pad 1: Net-(C47-Pad1) -> /I2C_SCL
- R1 pad 2: GND -> Net-(U3-SCL)
- R2 pad 1: Net-(Q1-G) -> /I2C_SDIO
- R2 pad 2: GND -> Net-(U3-SDA)
- R25 pad 1: Net-(U1-GPO1) -> Net-(U1-SDIO)
- R25 pad 2: +3V3 -> /I2C_SDIO
- R26 pad 1: Net-(U1-GPO2/INTB) -> Net-(U1-SCLK)
- R26 pad 2: GND -> /I2C_SCL
- R27 pad 1: Net-(U1-SDIO) -> Net-(U1-~{RST})
- R27 pad 2: /MCU_and_UI/I2C_SDIO -> /~{SI_RST}
- R28 pad 1: Net-(U1-SCLK) -> Net-(U1-GPO2/INTB)
- R28 pad 2: /MCU_and_UI/I2C_SCL -> GND
- R29 pad 1: Net-(U1-~{RST}) -> Net-(U1-GPO1)
- R29 pad 2: /MCU_and_UI/~{SI_RST} -> Net-(U1-VDD)
- R3 pad 1: /MCU_and_UI/RX_ant_en -> Net-(U4-TXD0/IO1)
- R3 pad 2: Net-(Q2-G) -> /ESP_TX
- R30 pad 1: Net-(U1-SENB) -> Net-(U6-IN_A+)
- R31 pad 1: Net-(U1-SENB) -> GND
- R31 pad 2: GND -> Net-(U6-IN_A+)
- R32 pad 1: /MCU_and_UI/I2C_SCL -> +3V3
- R32 pad 2: /TX/SCL -> Net-(U3-VDDO)
- R33 pad 1: /MCU_and_UI/I2C_SDIO -> Net-(C8-Pad1)
- R33 pad 2: /TX/SDA -> GND
- R34 pad 1: /MCU_and_UI/TX_Mod -> +3V3
- R34 pad 2: Net-(C55-Pad1) -> Net-(U8E-VCC)
- R35 pad 1: +3V3 -> /TX_Mod
- R35 pad 2: Net-(U3E-VCC) -> Net-(C21-Pad1)
- R4 pad 1: Net-(U2-IO12) -> Net-(U4-RXD0/IO3)
- R4 pad 2: GND -> /ESP_RX
- R40 pad 1: Net-(U4-D0) -> +3V3
- R40 pad 2: /MCU_and_UI/LCD.D0 -> /ESP_reset
- R41 pad 1: Net-(U4-D1) -> +3V3
- R41 pad 2: /MCU_and_UI/LCD.D1 -> Net-(C42-Pad2)
- R42 pad 1: Net-(U4-D2) -> +3V3
- R42 pad 2: /MCU_and_UI/LCD.D2 -> /PTT_key
- R43 pad 1: Net-(U4-D3) -> Net-(U4-IO2)
- R43 pad 2: /MCU_and_UI/LCD.D3 -> /RX_ant_en
- R44 pad 1: Net-(U4-D4) -> Net-(U4-IO12)
- R44 pad 2: /MCU_and_UI/LCD.D4 -> GND
- R45 pad 1: Net-(U4-D5) -> /mic_in
- R45 pad 2: /MCU_and_UI/LCD.D5 -> +3V3
- R46 pad 1: Net-(U4-D6) -> +3V3
- R46 pad 2: /MCU_and_UI/LCD.D6 -> /I2C_SCL
- R47 pad 1: Net-(U4-D7) -> +3V3
- R47 pad 2: /MCU_and_UI/LCD.D7 -> /I2C_SDIO
- R49 pad 1: GND -> /side_tone
- R49 pad 2: Net-(U4-Vss_backlight) -> /audio_out_right
- R51 pad 2: /MCU_and_UI/V_sense -> /V_sense
- R52 pad 1: /MCU_and_UI/V_sense -> /V_sense
- R53 pad 1: Net-(C55-Pad1) -> Net-(C21-Pad1)
- R54 pad 1: GND -> Net-(Q1-G)
- R54 pad 2: RF_GND -> GND
- R6 pad 2: /MCU_and_UI/onboard_mic -> /Encoder.btn
- R7 pad 1: /MCU_and_UI/mic_in -> Net-(C15-Pad2)
- R8 pad 1: /MCU_and_UI/side_tone -> /mic_in
- R8 pad 2: /MCU_and_UI/audio_out_right -> GND
- R9 pad 1: /MCU_and_UI/side_tone -> +3V3
- R9 pad 2: /MCU_and_UI/audio_out_left -> Net-(U3-VDD)
- SW7 pad 1: GND -> /onboard_key
- SW7 pad 2: /MCU_and_UI/Btn.Menu -> GND
- TP1 pad 1: /TX/Out2 -> Net-(U4-IO12)
- U1 pad 1: Net-(U1-LOUT/DFS) -> unconnected-(U1-LOUT/DFS-Pad1)
- U1 pad 10: Net-(U1-SENB) -> GND
- U1 pad 6: Net-(U1-FMI) -> unconnected-(U1-FMI-Pad6)
- U3 pad 1: Net-(U3-Pad1) -> Net-(U3-VDD)
- U3 pad 10: Net-(C47-Pad1) -> Net-(U3-CLK0)
- U3 pad 2: Net-(U3E-VCC) -> Net-(U3-XA)
- U3 pad 3: Net-(C8-Pad1) -> Net-(U3-XB)
- U3 pad 4: Net-(U3-Pad1) -> Net-(U3-SCL)
- U3 pad 5: Net-(U3E-VCC) -> Net-(U3-SDA)
- U3 pad 6: Net-(C8-Pad1) -> unconnected-(U3-CLK2-Pad6)
- U3 pad 7: GND -> Net-(U3-VDDO)
- U3 pad 8: Net-(U3-Pad1) -> GND
- U3 pad 9: Net-(U3E-VCC) -> unconnected-(U3-CLK1-Pad9)
- U4 pad 10: Net-(U4-D3) -> /TX_Mod
- U4 pad 11: Net-(U4-D4) -> /side_tone
- U4 pad 12: Net-(U4-D5) -> /Encoder.btn
- U4 pad 13: Net-(U4-D6) -> /V_sense
- U4 pad 14: Net-(U4-D7) -> Net-(U4-IO12)
- U4 pad 15: Net-(U4-Vdd_backlight) -> GND
- U4 pad 16: Net-(U4-Vss_backlight) -> /~{SI_RST}
- U4 pad 17: GND -> unconnected-(U4-NC-Pad17)
- U4 pad 18: GND -> unconnected-(U4-NC-Pad18)
- U4 pad 19: GND -> unconnected-(U4-NC-Pad19)
- U4 pad 2: Net-(U4-Chip_enable) -> Net-(U4-VDD)
- U4 pad 20: GND -> unconnected-(U4-NC-Pad20)
- U4 pad 3: Net-(U4-Vo) -> /ESP_reset
- U4 pad 4: Net-(U4-Data/~{Instruction}) -> unconnected-(U4-SENSOR_VP-Pad4)
- U4 pad 5: Net-(U4-R/~{L}) -> unconnected-(U4-SENSOR_VN-Pad5)
- U4 pad 6: Net-(U4-Chip_enable) -> /mic_in
- U4 pad 7: Net-(U4-D0) -> /PTT_key
- U4 pad 8: Net-(U4-D1) -> unconnected-(U4-IO32-Pad8)
- U4 pad 9: Net-(U4-D2) -> unconnected-(U4-IO33-Pad9)
Routing:
- net Net-(Q1-G): track 6.93 -> 66.8 mm, vias 0 -> 1
- net /ESP_boot: track 0.00 -> 46.8 mm, vias 0 -> 1
- net Net-(R7-Pad2): track 0.00 -> 45.2 mm, vias 0 -> 1
- net /audio_out_right: track 0.00 -> 40.6 mm, vias 0 -> 1
- net /Encoder.A: track 0.00 -> 39.5 mm, vias 0 -> 1
- net /Encoder.B: track 0.00 -> 39.3 mm, vias 0 -> 1
- net Net-(SW1C-C): track 38.6 -> 0.00 mm
- net Net-(U1-VDD): track 0.00 -> 38.6 mm, vias 0 -> 2
- net Net-(Q1-D): track 0.00 -> 38.0 mm
- net /I2C_SCL: track 0.00 -> 37.8 mm, vias 0 -> 3
- net /I2C_SDIO: track 0.00 -> 36.8 mm, vias 0 -> 3
- net Net-(SW1C-A): track 36.6 -> 0.00 mm
- net VBUS_filtered: track 0.00 -> 32.3 mm, vias 0 -> 9
- net /mic_in: track 0.00 -> 31.4 mm, vias 0 -> 2
- net /ESP_TX: track 0.00 -> 29.7 mm, vias 0 -> 1
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- added copper zone on In2.Cu, net +3V3
- added copper zone on In2.Cu, net +3V3_RX
- added copper zone on B.Cu, net GND
- added copper zone on In2.Cu, net Net-(U4-VDD)
- added copper zone on In2.Cu, net VBUS_filtered
- removed copper zone on F.Cu, net Net-(D5-K)
- removed copper zone on In1.Cu, net RF_GND
- removed copper zone on F.Cu, net VBUS
- removed copper zone on F.Cu, net VBUS_filtered
Other:
- board size 100 x 70 mm -> 78 x 47 mm
- board text added: "PCB size: 78mm x 47mm Uses 80x50x20 Case"
- board text added: "Summit Scourer MK1 Designed with love by ZL3APB"
- board text removed: "LCD contrast"

Commit message: Add files via upload
Parts:
- C11, C12, C25, C37, C39, C41, C46, C49, C61, C63, R44, R46, R47, R49, R51, R52, R6: moved to B.Cu
- moved R47 21.3 mm to (163.8, 101.1), turned to -90 degrees
- moved R46 21.2 mm to (163.8, 105.8), turned to 90 degrees
- moved C22 8.45 mm to (167.3, 84.5)
- moved C12 3.69 mm to (183.0, 104.7)
- moved C11 3.69 mm to (184.6, 104.7)
- moved J2 3.56 mm to (181.8, 110.7)
- moved C61 2.84 mm to (177.9, 103.8)
- moved R44 2.40 mm to (127.2, 97.6)
- moved R51 2.20 mm to (134.8, 96.7)
- moved R49 1.99 mm to (125.4, 105.5)
- moved R52 1.90 mm to (125.4, 103.0)
- moved C8 1.80 mm to (166.2, 97.0), turned to -90 degrees
- moved C49 1.70 mm to (181.7, 96.5), turned to 180 degrees
- moved C63 0.52 mm to (139.8, 96.8)
Routing:
- net Net-(Q1-D): track 38.0 -> 47.1 mm
- net Net-(Q1-G): track 66.8 -> 72.3 mm
- net Net-(C22-Pad1): track 18.5 -> 13.4 mm
- net VBUS_filtered: track 32.3 -> 28.7 mm, vias 9 -> 8
- net /V_sense: track 10.2 -> 13.0 mm, vias 1 -> 2
- net Net-(U3-CLK0): track 7.35 -> 4.55 mm
- net /mic_in: track 31.4 -> 34.0 mm
- net Net-(C8-Pad1): track 6.88 -> 8.29 mm
- net /audio_out_right: track 40.6 -> 39.3 mm, vias 1 -> 2
- net /side_tone: track 2.91 -> 1.78 mm, vias 1 -> 0
- net /I2C_SDIO: track 36.8 -> 35.9 mm
- net Net-(J2-In): track 6.83 -> 7.70 mm
- net /PTT_key: track 22.7 -> 23.5 mm, vias 0 -> 1
- net Net-(U4-IO12): track 6.38 -> 7.03 mm, vias 1 -> 0
- net +3V3: track 28.5 -> 27.9 mm
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