File: Kicad/_autosave-summit_scourer.kicad_pcb (KiCad board)
At the start: 2 copper layers, 100 x 70 mm, 150 parts, among them J1 SI5351_breakout_board, J2 Conn_Coaxial, J3 PTT/Mic, J4 Internal_SPK, J5 PTT/Mic, J6 RFShield_OnePiece, Q1 Q_NMOS, Q2 2N7002H, SW1 SW_DPDT_x3, SW2 push_btn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

Commit message: Add files via upload
Parts:
- moved T1 16.4 mm to (244.3, 55.8)
- moved T3 0.06 mm to (233.6, 55.8)
Routing:
- net Net-(D1-A): track 0.00 -> 16.8 mm
- net /channel_switching_and_filtering/RF_out: track 0.00 -> 6.74 mm
Changed lines of the file:
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@@
 	(footprint "summit_scourer:torroid_transformer"
 		(layer "F.Cu")
-		(at 233.565 55.74)
+		(at 233.565 55.8)
 		(descr "L_Toroid, Vertical series, Radial, pin pitch=5.08mm, , length*width=10*5mm^2")
 		(tags "L_Toroid Vertical series Radial pin pitch 5.08mm  length 10mm width 5mm")
@@
 	(footprint "summit_scourer:torroid_transformer"
 		(layer "F.Cu")
-		(at 233.565 43.38)
+		(at 244.3 55.8)
 		(descr "L_Toroid, Vertical series, Radial, pin pitch=5.08mm, , length*width=10*5mm^2")
 		(tags "L_Toroid Vertical series Radial pin pitch 5.08mm  length 10mm width 5mm")
 		(property "Reference" "T1"
-			(at 0 -2.25 0)
+			(at 0 -2.25 360)
 			(layer "F.SilkS")
 			(effects
@@
 		)
 		(property "Value" "T"
-			(at 0 7.33 0)
+			(at 0 7.33 360)
 			(layer "F.Fab")
 			(effects
@@
 		)
 		(fp_text user "${REFERENCE}"
-			(at 2.54 0 0)
+			(at 2.54 0 360)
 			(layer "F.Fab")
 			(effects
@@
 	)
 	(segment
+		(start 246.3 60.88)
+		(end 243.82 58.4)
+		(width 0.5)
+		(layer "F.Cu")
+		(net 46)
+	)
+	(segment
+		(start 234.165 58.4)
+		(end 231.565 55.8)
+		(width 0.5)
+		(layer "F.Cu")
+		(net 46)
+	)
+	(segment
+		(start 243.82 58.4)
+		(end 234.165 58.4)
+		(width 0.5)
+		(layer "F.Cu")
+		(net 46)
+	)
+	(segment
 		(start 102.5334 55.2)
 		(end 102.5334 53.333427)
@@
 	)
 	(segment
+		(start 235.565 55.8)
+		(end 242.3 55.8)
+		(width 0.5)
+		(layer "F.Cu")
+		(net 71)
+	)
+	(segment
