File: Kicad/channel_switching_and_filtering.kicad_sch (KiCad schematic)
At the start: 15 parts, among them SW1 SW_DPDT_x3

Commit message: Add files via upload
Parts:
- added C43, C44, C45, C46: 10n, Capacitor_SMD:C_0603_1608Metric_Pad1.08x0.95mm_HandSolder, symbol Device:C
- added D1, D2: D, Diode_SMD:D_PowerDI-123, symbol Device:D
- added R21, R22: 220R, Resistor_SMD:R_0603_1608Metric, symbol Device:R
- added R23, R24: 100k, Resistor_SMD:R_0603_1608Metric, symbol Device:R
- added T1, T3: T, symbol summit_scourer:Transformer_1P_1S_horizontal
- C20, C21, C22, C23, C24, C37, C38, C39, C40, C41: footprint (none) -> Capacitor_SMD:C_0603_1608Metric_Pad1.08x0.95mm_HandSolder
Connections:
- net GND: now also C43.2, C44.2, C45.2, C46.2, R21.2, R22.2, T1.3 (SA), T3.4 (SB)
- net at SW1.8 (B): now also T1.2 (AB)
- net TX_PA: now reaches SW1.5 (B)
- new net: C43.1, D2.1 (K), R23.1
- new net: D2.2 (A), R21.1, T3.2 (AB)
- new net: C44.1, D1.1 (K), R24.1
- new net: D1.2 (A), R22.1, T1.4 (SB), T3.1 (AA)
- new net Forward_indicator: C45.1, R23.2
- new net RF_out: T1.1 (AA), T3.3 (SA)
- new net Reverse_indicator: C46.1, R24.2
Other:
- moved on the sheet: C20, C21, C22, C23, C24, C37, C38, C39, C40, C41, L3, L4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

Commit message: Add files via upload
Parts:
- SW1: footprint (none) -> summit_scourer:SW_GF-161-0005
- T1, T3: footprint (none) -> summit_scourer:torroid_transformer
Changed lines of the file:
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@@
 			)
 		)
-		(property "Footprint" ""
+		(property "Footprint" "summit_scourer:SW_GF-161-0005"
 			(at 144.78 95.25 0)
 			(effects
@@
 			)
 		)
-		(property "Footprint" ""
+		(property "Footprint" "summit_scourer:torroid_transformer"
 			(at 171.45 116.84 90)
 			(effects
@@
 			)
 		)
-		(property "Footprint" ""
+		(property "Footprint" "summit_scourer:SW_GF-161-0005"
 			(at 54.61 95.25 0)
 			(effects
@@
 			)
 		)
-		(property "Footprint" ""
+		(property "Footprint" "summit_scourer:torroid_transformer"
 			(at 168.91 97.79 90)
 			(effects

Commit message: Add files via upload
Parts:
- removed C20, C21, C22, C23, C24, C37, C38, C39, C40, C41: C, Capacitor_SMD:C_0603_1608Metric_Pad1.08x0.95mm_HandSolder, symbol Device:C
- removed C43, C44, C45, C46: 10n, Capacitor_SMD:C_0603_1608Metric_Pad1.08x0.95mm_HandSolder, symbol Device:C
- removed D1, D2: D, Diode_SMD:D_PowerDI-123, symbol Device:D
- removed L3, L4, L6, L7: L_Ferrite, Inductor_THT:L_Toroid_Vertical_L10.0mm_W5.0mm_P5.08mm, symbol Device:L_Ferrite
- removed R21, R22: 220R, Resistor_SMD:R_0603_1608Metric, symbol Device:R
- removed R23, R24: 100k, Resistor_SMD:R_0603_1608Metric, symbol Device:R
- removed SW1: SW_DPDT_x3, summit_scourer:SW_GF-161-0005, symbol summit_scourer:SW_DPDT_x3
- removed T1, T3: T, summit_scourer:torroid_transformer, symbol summit_scourer:Transformer_1P_1S_horizontal
