File: Kicad/MCU_and_UI.kicad_sch (KiCad schematic)
At the start: 48 parts, among them J1 SI5351_breakout_board, J4 Audio_out, J5 Mic/Key, SW1 SW_DPDT_x3, SW2 PTT/Key, SW3 Up_key, SW4 Up_key, SW5 Up_key, SW6 Up_key, SW7 Up_key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

Commit message: Add files via upload
Parts:
- removed C3: 10n, Capacitor_SMD:C_0603_1608Metric_Pad1.08x0.95mm_HandSolder, symbol Device:C
- removed C4: 100n, Capacitor_SMD:C_0504_1310Metric_Pad0.83x1.28mm_HandSolder, symbol Device:C
- removed C5: 10u, Capacitor_SMD:C_1210_3225Metric_Pad1.33x2.70mm_HandSolder, symbol Device:C
- removed J1: SI5351_breakout_board, Connector_PinHeader_2.54mm:PinHeader_1x07_P2.54mm_Vertical, symbol Connector:Conn_01x07_Pin
- removed RV1: 10k, symbol Device:R_Potentiometer_Trim
- added R36: 0R, summit_scourer:R_0603_linked, symbol Device:R
- added R37: 10k, Resistor_SMD:R_0603_1608Metric, symbol Device:R
- C25, C27, C30, C31: footprint Capacitor_SMD:C_0504_1310Metric_Pad0.83x1.28mm_HandSolder -> Capacitor_SMD:C_0603_1608Metric_Pad1.08x0.95mm_HandSolder
- J4, J5: footprint (none) -> Connector_Audio:Jack_3.5mm_CUI_SJ1-3525N_Horizontal
- L5: footprint (none) -> Inductor_THT:L_Toroid_Vertical_L10.0mm_W5.0mm_P5.08mm
- R10, R13, R14, R15, R16, R17, R20, R4, R5, R6, R8, R9: footprint (none) -> Resistor_SMD:R_0603_1608Metric
- R11, R7: footprint (none) -> summit_scourer:R_0603_linked
- R12: value 0R -> 10k; footprint (none) -> Resistor_SMD:R_0603_1608Metric; now fitted; now in the parts list
- R18, R19: value 10k -> 1k; footprint (none) -> Resistor_SMD:R_0603_1608Metric
- SW2: value PTT/Key -> push_btn; footprint (none) -> Button_Switch_SMD:SW_Push_1P1T_NO_6x6mm_H9.5mm
- SW3, SW4, SW5, SW6, SW7: value Up_key -> push_btn; footprint (none) -> Button_Switch_SMD:SW_Push_1P1T_NO_6x6mm_H9.5mm
- U4: footprint (none) -> summit_scourer:Display_8x2
Connections:
- net +3V3: now also R37.1
- net GND: now also R12.2, U4.17, U4.18, U4.19, U4.20
- net at C31.1, R11.2, U4.2 (Vdd)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: no longer R12.2
- net at U4.3 (Vo): now also R12.1, R37.2
- net ~{SI_RST}: now reaches U2.16 (IO13)
- net at U2.24 (IO2): now also R36.1
- net SCL renamed I2C_SDIO
- net SDA renamed I2C_SCL
- new net RX_ant_en: R36.2
Other:
- note added: "Contrast setting"
- moved on the sheet: C31, C32, C33, C34, C35, C36, R11, R13, R14, R15, R16, R17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

Commit message: Add files via upload
Parts:
- added C51: 10u, Capacitor_SMD:C_1210_3225Metric_Pad1.33x2.70mm_HandSolder, symbol Device:C
- added R38, R39, R40, R41, R42, R43, R44, R45, R46, R47, R48, R49: 0R, summit_scourer:R_0603_linked, symbol Device:R
- L5: footprint Inductor_THT:L_Toroid_Vertical_L10.0mm_W5.0mm_P5.08mm -> Inductor_SMD:L_TDK_SLF6025
- SW1: footprint (none) -> summit_scourer:SW_GF-161-0005
- SW2, SW3, SW4, SW5, SW6, SW7: footprint Button_Switch_SMD:SW_Push_1P1T_NO_6x6mm_H9.5mm -> Button_Switch_THT:SW_PUSH_6mm_H9.5mm
Connections:
- net GND: now also C51.2, R49.1; no longer U4.16 (Vss_backlight)
- net LCD.BL: now also R48.1; no longer U4.15 (Vdd_backlight)
- net LCD.D0: now also R40.2; no longer U4.7 (D0)
- net LCD.D1: now also R41.2; no longer U4.8 (D1)
- net LCD.D2: now also R42.2; no longer U4.9 (D2)
- net LCD.D3: now also R43.2; no longer U4.10 (D3)
- net LCD.D4: now also R44.2; no longer U4.11 (D4)
- net LCD.D5: now also R45.2; no longer U4.12 (D5)
- net LCD.D6: now also R46.2; no longer U4.13 (D6)
- net LCD.D7: now also R47.2; no longer U4.14 (D7)
- net LCD.D/I: now also R38.2; no longer U4.4 (Data/~{Instruction})
- net LCD.R/L: now also R39.2; no longer U4.5 (R/~{L})
- net at C25.1, C26.1, L5.1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: now also C51.1
- new net: R45.1, U4.12 (D5)
- new net: R41.1, U4.8 (D1)
- new net: R48.2, U4.15 (Vdd_backlight)
- new net: R38.1, U4.4 (Data/~{Instruction})
- new net: R43.1, U4.10 (D3)
- new net: R44.1, U4.11 (D4)
- new net: R46.1, U4.13 (D6)
- new net: R47.1, U4.14 (D7)
- new net: R49.2, U4.16 (Vss_backlight)
- new net: R39.1, U4.5 (R/~{L})
- new net: R40.1, U4.7 (D0)
- new net: R42.1, U4.9 (D2)
Other:
- moved on the sheet: C26

Commit message: Add files via upload
Parts:
- removed J4: Audio_out, Connector_Audio:Jack_3.5mm_CUI_SJ1-3525N_Horizontal, symbol Connector_Audio:AudioJack2_Ground
- removed J5: Mic/Key, Connector_Audio:Jack_3.5mm_CUI_SJ1-3525N_Horizontal, symbol Connector_Audio:AudioJack2_Ground_Switch
- added J3, J5: PTT/Mic, Connector_Audio:Jack_3.5mm_CUI_SJ1-3525N_Horizontal, symbol summit_scourer:AudioJack2_Ground_Switch
- added J4: Internal_SPK, Connector_PinHeader_2.54mm:PinHeader_1x03_P2.54mm_Vertical, symbol Connector:Conn_01x03_Pin
- added R51: 100k, Resistor_SMD:R_0603_1608Metric, symbol Device:R
- added R52: 10k, Resistor_SMD:R_0603_1608Metric, symbol Device:R
Connections:
- net GND: now also J3.S, J4.3 (Pin_3), J5.S, R52.2
- net PTT_key: now also J3.T
- net audio_out_left: now also J5.T
- net audio_out_right: now also J5.R
- net onboard_key: now also J3.TN
- net onboard_mic: now also J3.RN
- net V_sense: now reaches U2.13 (IO14)
- net V_sense: now also R51.2, R52.1
- net at C30.2: now also J3.R
- new net: J4.1 (Pin_1), J5.RN
- new net: J4.2 (Pin_2), J5.TN
- new net VBUS_filtered: R51.1

Commit message: Add files via upload
Parts:
- added TP3: IO12, Connector_PinHeader_2.54mm:PinHeader_1x01_P2.54mm_Vertical, symbol Connector:TestPoint
- MK1: footprint (none) -> Connector_PinHeader_2.54mm:PinHeader_1x02_P2.54mm_Vertical
Connections:
- net LCD.BL: now also U2.27 (IO16); no longer U2.10 (IO25)
- net at R4.1, U2.14 (IO12): now also TP3.1
- new net TX_Mod: U2.10 (IO25)
Other:
- moved on the sheet: R36
Changed lines of the file:
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@@
 	)
 	(junction
+		(at 180.34 68.58)
+		(diameter 0)
+		(color 0 0 0 0)
+	)
+	(junction
 		(at 168.91 151.13)
 		(diameter 0)
@@
 	)
 	(bus_entry
-		(at 179.07 93.98)
+		(at 179.07 76.2)
 		(size -2.54 2.54)
 		(stroke
@@
 	(wire
 		(pts
-			(xy 167.64 68.58) (xy 184.15 68.58)
+			(xy 167.64 68.58) (xy 180.34 68.58)
 		)
 		(stroke
@@
 	(wire
 		(pts
+			(xy 181.61 76.2) (xy 233.68 76.2)
+		)
+		(stroke
+			(width 0)
+			(type default)
+		)
+	)
+	(wire
+		(pts
 			(xy 55.88 67.31) (xy 50.8 67.31)
 		)
@@
 	(wire
 		(pts
+			(xy 180.34 48.26) (xy 180.34 68.58)
+		)
+		(stroke
+			(width 0)
+			(type default)
+		)
+	)
+	(wire
+		(pts
 			(xy 74.93 31.75) (xy 74.93 33.02)
 		)
@@
 	(wire
 		(pts
+			(xy 167.64 96.52) (xy 196.85 96.52)
+		)
+		(stroke
+			(width 0)
+			(type default)
+		)
+	)
+	(wire
+		(pts
 			(xy 167.64 99.06) (xy 212.09 99.06)
 		)
@@
 	(wire
 		(pts
+			(xy 175.26 76.2) (xy 175.26 74.93)
+		)
+		(stroke
+			(width 0)
+			(type default)
+		)
+	)
+	(wire
+		(pts
 			(xy 233.68 107.95) (xy 233.68 76.2)
 		)
@@
 	(wire
 		(pts
-			(xy 177.8 58.42) (xy 182.88 58.42)
+			(xy 179.07 58.42) (xy 182.88 58.42)
 		)
 		(stroke
@@
 	(wire
 		(pts
+			(xy 184.15 91.44) (xy 184.15 104.14)
+		)
+		(stroke
+			(width 0)
+			(type default)
+		)
+	)
+	(wire
+		(pts
 			(xy 214.63 53.34) (xy 214.63 52.07)
 		)
@@
 		)
 	)
-	(bus
-		(pts
-			(xy 179.07 91.44) (xy 179.07 93.98)
-		)
-		(stroke
-			(width 0)
-			(type default)
-		)
-	)
 	(wire
 		(pts
@@
 	(wire
 		(pts
-			(xy 233.68 76.2) (xy 167.64 76.2)
-		)
-		(stroke
-			(width 0)
-			(type default)
-		)
-	)
-	(wire
-		(pts
 			(xy 50.8 119.38) (xy 45.72 119.38)
 		)
@@
 	(wire
 		(pts
+			(xy 167.64 76.2) (xy 175.26 76.2)
+		)
+		(stroke
+			(width 0)
+			(type default)
+		)
+	)
+	(wire
+		(pts
 			(xy 36.83 104.14) (xy 36.83 106.68)
 		)
@@
 	(wire
 		(pts
-			(xy 167.64 58.42) (xy 170.18 58.42)
+			(xy 167.64 58.42) (xy 171.45 58.42)
 		)
 		(stroke
@@
 		)
 	)
+	(bus
+		(pts
+			(xy 179.07 76.2) (xy 179.07 78.74)
+		)
+		(stroke
+			(width 0)
+			(type default)
+		)
+	)
 	(wire
 		(pts
@@
 	(wire
 		(pts
-			(xy 176.53 96.52) (xy 167.64 96.52)
+			(xy 176.53 78.74) (xy 167.64 78.74)
 		)
 		(stroke
@@
 	(wire
 		(pts
+			(xy 175.26 74.93) (xy 181.61 74.93)
+		)
+		(stroke
+			(width 0)
+			(type default)
+		)
+	)
+	(wire
+		(pts
+			(xy 182.88 48.26) (xy 180.34 48.26)
+		)
+		(stroke
+			(width 0)
+			(type default)
+		)
+	)
+	(wire
+		(pts
 			(xy 31.75 67.31) (xy 43.18 67.31)
 		)
@@
 	(bus
 		(pts
-			(xy 179.07 93.98) (xy 179.07 127)
+			(xy 179.07 91.44) (xy 179.07 127)
 		)
 		(stroke
@@
 	(wire
 		(pts
+			(xy 180.34 68.58) (xy 184.15 68.58)
+		)
+		(stroke
+			(width 0)
+			(type default)
+		)
+	)
+	(wire
+		(pts
 			(xy 256.54 73.66) (xy 256.54 72.39)
 		)
@@
 	(wire
 		(pts
-			(xy 184.15 104.14) (xy 184.15 91.44)
+			(xy 181.61 74.93) (xy 181.61 76.2)
 		)
 		(stroke
@@
 	)
 	(label "Band_select"
-		(at 168.91 76.2 0)
+		(at 181.61 76.2 0)
 		(fields_autoplaced yes)
 		(effects
@@
 	)
 	(label "LCD.BL"
-		(at 176.53 96.52 180)
+		(at 176.53 78.74 180)
 		(fields_autoplaced yes)
 		(effects
@@
 		)
 	)
+	(hierarchical_label "TX_Mod"
+		(shape input)
+		(at 196.85 96.52 0)
+		(fields_autoplaced yes)
+		(effects
+			(font
+				(size 1.27 1.27)
+			)
+			(justify left)
+		)
+	)
 	(symbol
 		(lib_id "Device:R")
@@
 	)
 	(symbol
+		(lib_id "Connector:TestPoint")
+		(at 182.88 48.26 270)
+		(unit 1)
+		(exclude_from_sim no)
+		(in_bom yes)
+		(on_board yes)
+		(dnp no)
+		(fields_autoplaced yes)
+		(property "Reference" "TP3"
+			(at 187.96 46.9899 90)
+			(effects
+				(font
+					(size 1.27 1.27)
+				)
+				(justify left)
+			)
+		)
+		(property "Value" "IO12"
+			(at 187.96 49.5299 90)
+			(effects
+				(font
+					(size 1.27 1.27)
+				)
+				(justify left)
+			)
+		)
+		(property "Footprint" "Connector_PinHeader_2.54mm:PinHeader_1x01_P2.54mm_Vertical"
+			(at 182.88 53.34 0)
+			(effects
+				(font
+					(size 1.27 1.27)
+				)
+				(hide yes)
+			)
+		)
+		(property "Datasheet" "~"
+			(at 182.88 53.34 0)
+			(effects
+				(font
+					(size 1.27 1.27)
+				)
+				(hide yes)
+			)
+		)
+		(property "Description" "test point"
+			(at 182.88 48.26 0)
+			(effects
+				(font
+					(size 1.27 1.27)
+				)
+				(hide yes)
+			)
+		)
+		(pin "1"
+		)
+		(instances
+			(project "summit_scourer"
+				(path "/97fa5a9e-fea2-40ae-976c-23c41ffbf522/9c59661f-2506-4efd-9bc6-e2f1b812693d"
+					(reference "TP3")
+					(unit 1)
+				)
+			)
+		)
+	)
+	(symbol
 		(lib_id "power:GND1")
 		(at 26.67 77.47 0)
@@
 	(symbol
 		(lib_id "Device:R")
-		(at 173.99 58.42 90)
+		(at 175.26 58.42 90)
 		(unit 1)
 		(exclude_from_sim no)
@@
 		(dnp no)
 		(property "Reference" "R36"
-			(at 178.816 57.404 90)
+			(at 170.434 57.404 90)
 			(effects
 				(font
@@
 		)
 		(property "Value" "0R"
-			(at 173.99 58.42 90)
+			(at 175.26 58.42 90)
 			(effects
 				(font
@@
 		)
 		(property "Footprint" "summit_scourer:R_0603_linked"
-			(at 173.99 60.198 90)
+			(at 175.26 60.198 90)
 			(effects
 				(font
@@
 		)
 		(property "Datasheet" "~"
-			(at 173.99 58.42 0)
+			(at 175.26 58.42 0)
 			(effects
 				(font
@@
 		)
 		(property "Description" "Resistor"
-			(at 173.99 58.42 0)
+			(at 175.26 58.42 0)
 			(effects
 				(font
@@
 			)
 		)
-		(property "Footprint" ""
+		(property "Footprint" "Connector_PinHeader_2.54mm:PinHeader_1x02_P2.54mm_Vertical"
 			(at 133.35 184.15 90)
 			(effects

Commit message: Add files via upload
Parts:
- removed C25, C27, C29, C30, C31, C32, C33, C34, C35, C36, C42: 100n, Capacitor_SMD:C_0603_1608Metric_Pad1.08x0.95mm_HandSolder, symbol Device:C
- removed C26, C28: 10n, Capacitor_SMD:C_0603_1608Metric_Pad1.08x0.95mm_HandSolder, symbol Device:C
- removed C51: 10u, Capacitor_SMD:C_1210_3225Metric_Pad1.33x2.70mm_HandSolder, symbol Device:C
- removed J3, J5: PTT/Mic, Connector_Audio:Jack_3.5mm_CUI_SJ1-3525N_Horizontal, symbol summit_scourer:AudioJack2_Ground_Switch
- removed J4: Internal_SPK, Connector_PinHeader_2.54mm:PinHeader_1x03_P2.54mm_Vertical, symbol Connector:Conn_01x03_Pin
- removed L5: L_Ferrite, Inductor_SMD:L_TDK_SLF6025, symbol Device:L_Ferrite
- removed MK1: Microphone, Connector_PinHeader_2.54mm:PinHeader_1x02_P2.54mm_Vertical, symbol Device:Microphone
- removed R10, R12, R13, R14, R15, R16, R17, R20, R37, R4, R52, R6, R8, R9: 10k, Resistor_SMD:R_0603_1608Metric, symbol Device:R
- removed R11, R36, R38, R39, R40, R41, R42, R43, R44, R45, R46, R47, R48, R49, R7: 0R, summit_scourer:R_0603_linked, symbol Device:R
- removed R18, R19: 1k, Resistor_SMD:R_0603_1608Metric, symbol Device:R
- removed R5, R51: 100k, Resistor_SMD:R_0603_1608Metric, symbol Device:R
- removed SW1: SW_DPDT_x3, summit_scourer:SW_GF-161-0005, symbol summit_scourer:SW_DPDT_x3
- removed SW2, SW3, SW4, SW5, SW6, SW7: push_btn, Button_Switch_THT:SW_PUSH_6mm_H9.5mm, symbol Switch:SW_SPST
- removed TP3: IO12, Connector_PinHeader_2.54mm:PinHeader_1x01_P2.54mm_Vertical, symbol Connector:TestPoint
- removed U2: ESP32-WROOM-32UE, RF_Module:ESP32-WROOM-32UE, symbol RF_Module:ESP32-WROOM-32UE
- removed U4: ~, summit_scourer:Display_8x2, symbol summit_scourer:8x2_LCD
Connections:
- no-connect marks 1 -> 0
Other:
- note removed: "Contrast setting"
- note removed: "ESP32 Input only pins: Name Num Sensor_VP 4 Sensor_VN 5 IO34 6 IO35 7 DAC pins: Name Num DAC name IO24 10 DAC_1 IO26 11 DAC_2"
