File: Kicad/PSU.kicad_sch (KiCad schematic)
At the start: 15 parts, among them U5 AZ1117-3.3, U6 AZ1117-5.0, U7 AZ1117-3.3

Commit message: Add files via upload
Parts:
- removed C53, C55: 10u, Capacitor_SMD:C_1210_3225Metric_Pad1.33x2.70mm_HandSolder, symbol Device:C
- removed U6: AZ1117-5.0, Package_TO_SOT_SMD:TO-252-2, symbol Regulator_Linear:AZ1117-3.3
Connections:
- net +5V is gone; now on net VBUS_filtered: C54.1, C56.1, U5.3 (VI), U7.3 (VI)
- net VBUS_filtered: now reaches C58.1, L9.2

Commit message: Add files via upload
Parts:
- added D5: 1N4007, Diode_THT:D_A-405_P2.54mm_Vertical_AnodeUp, symbol Device:D
Connections:
- net VBUS: now also D5.2 (A); no longer L9.1
- new net: D5.1 (K), L9.1
Other:
- moved on the sheet: C52, C56, C57, C58, C59, H1, H2, L9, R50, U7

Commit message: Add files via upload
Parts:
- removed C52, C54, C56, C57: 10u, Capacitor_SMD:C_1210_3225Metric_Pad1.33x2.70mm_HandSolder, symbol Device:C
- removed C58: 470u, Capacitor_THT:CP_Radial_D8.0mm_P3.80mm, symbol Device:C_Polarized
- removed C59: 100n, Capacitor_SMD:C_0603_1608Metric_Pad1.08x0.95mm_HandSolder, symbol Device:C
- removed D5: 1N4007, Diode_THT:D_A-405_P2.54mm_Vertical_AnodeUp, symbol Device:D
- removed H1: Vin_+, TestPoint:TestPoint_THTPad_3.0x3.0mm_Drill1.5mm, symbol Mechanical:MountingHole_Pad
- removed H2: Vin_-, TestPoint:TestPoint_THTPad_3.0x3.0mm_Drill1.5mm, symbol Mechanical:MountingHole_Pad
- removed L9: L_Ferrite, Inductor_SMD:L_6.3x6.3_H3, symbol Device:L_Ferrite
- removed R50: 0R, summit_scourer:R_0603_linked, symbol Device:R
- removed U5, U7: AZ1117-3.3, Package_TO_SOT_SMD:TO-252-2, symbol Regulator_Linear:AZ1117-3.3
