File: Kicad/TX.kicad_sch (KiCad schematic)
At the start: 10 parts, among them Q1 Q_NMOS, U3 74AC00

Commit message: Add files via upload
Parts:
- added C3: 10u, Capacitor_SMD:C_1210_3225Metric_Pad1.33x2.70mm_HandSolder, symbol Device:C
- added C4, C47: 100n, Capacitor_SMD:C_0603_1608Metric_Pad1.08x0.95mm_HandSolder, symbol Device:C
- added C5: 10n, Capacitor_SMD:C_0603_1608Metric_Pad1.08x0.95mm_HandSolder, symbol Device:C
- added J1: SI5351_breakout_board, Connector_PinHeader_2.54mm:PinHeader_1x07_P2.54mm_Vertical, symbol Connector:Conn_01x07_Pin
- added R32, R33, R34, R35: 0R, summit_scourer:R_0603_linked, symbol Device:R
- added RV1: 10k, Resistor_SMD:R_0603_1608Metric, symbol Device:R_Potentiometer_Trim
- C14, C6: footprint Capacitor_SMD:C_0504_1310Metric_Pad0.83x1.28mm_HandSolder -> Capacitor_SMD:C_0603_1608Metric_Pad1.08x0.95mm_HandSolder
- L1: footprint (none) -> Inductor_THT:L_Toroid_Vertical_L10.0mm_W5.0mm_P5.08mm
- R1, R2: footprint (none) -> Resistor_SMD:R_0603_1608Metric
- U3: footprint (none) -> Package_SO:SOIC-14_3.9x8.7mm_P1.27mm
Connections:
- net +5V: now also R34.1; no longer C6.1, C7.1, U3.13, U3.14 (VCC), U3.2, U3.5, U3.9
- net GND: now also C3.2, C4.2, C5.2, J1.2 (Pin_2)
- net VBUS: now reaches C14.1, L1.1
- net at C9.1, R1.1, U3.10: now also C47.1
- new net: C6.1, C7.1, R34.2, R35.2, U3.13, U3.14 (VCC), U3.2, U3.5, U3.9
- new net +3V3: C3.1, C4.1, C5.1, J1.1 (Pin_1), R35.1
- new net I2C_SCL: R32.1
- new net I2C_SDIO: R33.1
- new net Out1: C47.2, J1.5 (Pin_5)
- new net Out2: J1.6 (Pin_6), RV1.1
- new net Out3: J1.7 (Pin_7)
- new net RX_BFO: RV1.2, RV1.3
- new net SCL: J1.3 (Pin_3), R32.2
- new net SDA: J1.4 (Pin_4), R33.2
Other:
- moved on the sheet: C14, C6, C7, C8, C9, L1, Q1, R1, R2, U3A, U3B, U3C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

Commit message: Add files via upload
Parts:
- removed R34: 0R, summit_scourer:R_0603_linked, symbol Device:R
- removed RV1: 10k, Resistor_SMD:R_0603_1608Metric, symbol Device:R_Potentiometer_Trim
- added C53: 10u, Capacitor_SMD:C_1210_3225Metric, symbol Device:C
- added TP1: RX_BFO, TestPoint:TestPoint_THTPad_1.5x1.5mm_Drill0.7mm, symbol Connector:TestPoint
Connections:
- net GND: now also C53.2
- net Out2: now also TP1.1
- net VBUS renamed VBUS_filtered
- net VBUS_filtered: now also C53.1
Other:
- moved on the sheet: C14, C8

Commit message: Add files via upload
Parts:
- added C20, C21, C22, C23, C24, C37, C38, C39, C40, C41: C, Capacitor_SMD:C_0603_1608Metric_Pad1.08x0.95mm_HandSolder, symbol Device:C
- added C55: 10n, Capacitor_SMD:C_0603_1608Metric_Pad1.08x0.95mm_HandSolder, symbol Device:C
- added L3, L4, L6, L7: L_Ferrite, Inductor_THT:L_Toroid_Vertical_L10.0mm_W5.0mm_P5.08mm, symbol Device:L_Ferrite
- added R34, R53: 10k, Resistor_SMD:R_0603_1608Metric, symbol Device:R
- added SW1: SW_DPDT_x3, summit_scourer:SW_GF-161-0005, symbol summit_scourer:SW_DPDT_x3
Connections:
- net GND: now also C55.2
- net TX_PA: now also SW1.5 (B)
- net at C8.2, Q1.1 (G), R2.1: now also R53.2
- net VBUS_filtered renamed VBUS
- new net: C55.1, R34.2, R53.1
- new net: C21.1, C23.1, SW1.6 (C)
- new net: C23.2, L4.1
- new net: C24.2, C38.1, L3.2, L6.1
- new net: C38.2, C40.1, L6.2, SW1.7 (A)
- new net: C20.1, C22.1, SW1.4 (A)
- new net: C22.2, L3.1
- new net: C39.2, C41.1, L7.2, SW1.9 (C)
- new net: C37.2, C39.1, L4.2, L7.1
- new net RF_GND: C20.2, C21.2, C24.1, C37.1, C40.2, C41.2
- new net RF_out: SW1.8 (B)
- new net TX_Mod: R34.1
Other:
- moved on the sheet: C14, C3, C4, C47, C5, C53, C6, C7, C8, C9, L1, Q1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

Commit message: Add files via upload
Other:
- moved on the sheet: U3A
Changed lines of the file:
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@@
+	)
+	(junction
+		(at 90.17 116.84)
+		(diameter 0)
+		(color 0 0 0 0)
 	)
 	(junction
@@
 	)
 	(junction
-		(at 111.76 120.65)
-		(diameter 0)
-		(color 0 0 0 0)
-	)
-	(junction
 		(at 163.83 100.33)
 		(diameter 0)
@@
 	)
 	(junction
-		(at 90.17 118.11)
-		(diameter 0)
-		(color 0 0 0 0)
-	)
-	(junction
 		(at 226.06 80.01)
 		(diameter 0)
@@
 	)
 	(junction
+		(at 111.76 119.38)
+		(diameter 0)
+		(color 0 0 0 0)
+	)
+	(junction
 		(at 46.99 74.93)
 		(diameter 0)
@@
 	)
 	(junction
-		(at 92.71 123.19)
+		(at 92.71 121.92)
 		(diameter 0)
 		(color 0 0 0 0)
@@
 	(wire
 		(pts
+			(xy 111.76 119.38) (xy 111.76 133.35)
+		)
+		(stroke
+			(width 0)
+			(type default)
+		)
+	)
+	(wire
+		(pts
 			(xy 64.77 127) (xy 67.31 127)
 		)
@@
 	(wire
 		(pts
+			(xy 90.17 116.84) (xy 90.17 130.81)
+		)
+		(stroke
+			(width 0)
+			(type default)
+		)
+	)
+	(wire
+		(pts
 			(xy 62.23 72.39) (xy 62.23 67.31)
 		)
@@
 	(wire
 		(pts
-			(xy 111.76 120.65) (xy 109.22 120.65)
+			(xy 111.76 119.38) (xy 109.22 119.38)
 		)
 		(stroke
@@
 	(wire
 		(pts
-			(xy 111.76 107.95) (xy 111.76 120.65)
+			(xy 111.76 107.95) (xy 111.76 119.38)
 		)
 		(stroke
@@
 	(wire
 		(pts
-			(xy 92.71 123.19) (xy 92.71 135.89)
-		)
-		(stroke
-			(width 0)
-			(type default)
-		)
-	)
-	(wire
-		(pts
 			(xy 69.85 114.3) (xy 69.85 100.33)
 		)
@@
 	(wire
 		(pts
-			(xy 92.71 123.19) (xy 93.98 123.19)
+			(xy 92.71 121.92) (xy 93.98 121.92)
 		)
 		(stroke
@@
 	(wire
 		(pts
-			(xy 90.17 118.11) (xy 93.98 118.11)
-		)
-		(stroke
-			(width 0)
-			(type default)
-		)
-	)
-	(wire
-		(pts
-			(xy 111.76 133.35) (xy 111.76 120.65)
+			(xy 90.17 116.84) (xy 93.98 116.84)
 		)
 		(stroke
@@
 	(wire
 		(pts
-			(xy 92.71 107.95) (xy 92.71 123.19)
+			(xy 92.71 107.95) (xy 92.71 121.92)
 		)
 		(stroke
@@
 	(wire
 		(pts
-			(xy 90.17 118.11) (xy 90.17 130.81)
+			(xy 92.71 121.92) (xy 92.71 135.89)
 		)
 		(stroke
@@
 	(wire
 		(pts
-			(xy 90.17 111.76) (xy 90.17 118.11)
+			(xy 90.17 111.76) (xy 90.17 116.84)
 		)
 		(stroke
@@
 	(symbol
 		(lib_id "74xx:74HC00")
-		(at 101.6 120.65 0)
+		(at 101.6 119.38 0)
 		(unit 1)
 		(exclude_from_sim no)
@@
 		(dnp no)
 		(property "Reference" "U3"
-			(at 101.346 120.65 0)
+			(at 101.346 119.38 0)
 			(effects
 				(font
@@
 		)
 		(property "Value" "74AC00"
-			(at 101.6 115.57 0)
+			(at 101.6 114.3 0)
 			(effects
 				(font
@@
 		)
 		(property "Footprint" "Package_SO:SOIC-14_3.9x8.7mm_P1.27mm"
-			(at 101.6 120.65 0)
+			(at 101.6 119.38 0)
 			(effects
 				(font
@@
 		)
 		(property "Datasheet" ""
-			(at 101.6 120.65 0)
+			(at 101.6 119.38 0)
 			(effects
 				(font
@@
 		)
 		(property "Description" "quad 2-input NAND gate"
-			(at 101.6 120.65 0)
-			(effects
-				(font
+			(at 101.6 119.38 0)
+			(effects
+				(font

Commit message: Add files via upload
Parts:
- removed C14, C4, C47, C6: 100n, Capacitor_SMD:C_0603_1608Metric_Pad1.08x0.95mm_HandSolder, symbol Device:C
- removed C20, C21, C22, C23, C24, C37, C38, C39, C40, C41: C, Capacitor_SMD:C_0603_1608Metric_Pad1.08x0.95mm_HandSolder, symbol Device:C
- removed C3: 10u, Capacitor_SMD:C_1210_3225Metric_Pad1.33x2.70mm_HandSolder, symbol Device:C
- removed C5, C55, C7, C8: 10n, Capacitor_SMD:C_0603_1608Metric_Pad1.08x0.95mm_HandSolder, symbol Device:C
- removed C53: 10u, Capacitor_SMD:C_1210_3225Metric, symbol Device:C
- removed C9: 22p, Capacitor_SMD:C_0603_1608Metric_Pad1.08x0.95mm_HandSolder, symbol Device:C
- removed J1: SI5351_breakout_board, Connector_PinHeader_2.54mm:PinHeader_1x07_P2.54mm_Vertical, symbol Connector:Conn_01x07_Pin
- removed L1: L, Inductor_THT:L_Toroid_Vertical_L10.0mm_W5.0mm_P5.08mm, symbol Device:L
- removed L3, L4, L6, L7: L_Ferrite, Inductor_THT:L_Toroid_Vertical_L10.0mm_W5.0mm_P5.08mm, symbol Device:L_Ferrite
- removed Q1: Q_NMOS, Package_TO_SOT_SMD:SOT-89-3_Handsoldering, symbol Device:Q_NMOS_GSD
- removed R1, R2: 100k, Resistor_SMD:R_0603_1608Metric, symbol Device:R
- removed R32, R33, R35: 0R, summit_scourer:R_0603_linked, symbol Device:R
- removed R34, R53: 10k, Resistor_SMD:R_0603_1608Metric, symbol Device:R
- removed SW1: SW_DPDT_x3, summit_scourer:SW_GF-161-0005, symbol summit_scourer:SW_DPDT_x3
- removed TP1: RX_BFO, TestPoint:TestPoint_THTPad_1.5x1.5mm_Drill0.7mm, symbol Connector:TestPoint
- removed U3: 74AC00, Package_SO:SOIC-14_3.9x8.7mm_P1.27mm, symbol 74xx:74HC00
