File: Kicad/summit_scourer.kicad_sch (KiCad schematic)
At the start: 3 parts, among them J2 Conn_Coaxial

Commit message: Add files via upload
Parts:
- C11, C12: footprint Capacitor_SMD:C_0504_1310Metric_Pad0.83x1.28mm_HandSolder -> Capacitor_SMD:C_0603_1608Metric_Pad1.08x0.95mm_HandSolder
- J2: footprint (none) -> Connector_Coaxial:SMA_Amphenol_901-143_Horizontal
Other:
- sheet MCU_and_UI ports: added ESP_RX, ESP_TX, ESP_boot, ESP_reset, I2C_SCL, I2C_SDIO, RX_ant_en, TX_LO, audio_out_left, audio_out_right, ~{SI_RST}; removed none
- sheet RX ports: added I2C_SCL, I2C_SDIO, audio_out_left, audio_out_right, ~{SI_RST}; removed none
- sheet TX ports: added I2C_SCL, I2C_SDIO, RX_BFO; removed TX_VFO
- sheet channel_switching_and_filtering ports: added Forward_indicator, RF_out, Reverse_indicator, TX_PA; removed none

Commit message: Add files via upload
Other:
- added sheet PSU (PSU.kicad_sch)
Changed lines of the file:
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@@
+	)
+	(sheet
+		(at 64.516 21.844)
+		(size 40.894 19.05)
+		(fields_autoplaced yes)
+		(stroke
+			(width 0.1524)
+			(type solid)
+		)
+		(fill
+			(color 0 0 0 0.0000)
+		)
+		(property "Sheetname" "PSU"
+			(at 64.516 21.1324 0)
+			(effects
+				(font
+					(size 1.27 1.27)
+				)
+				(justify left bottom)
+			)
+		)
+		(property "Sheetfile" "PSU.kicad_sch"
+			(at 64.516 41.4786 0)
+			(effects
+				(font
+					(size 1.27 1.27)
+				)
+				(justify left top)
+			)
+		)
+		(instances
+			(project "summit_scourer"
+				(path "/97fa5a9e-fea2-40ae-976c-23c41ffbf522"
+					(page "6")
+				)
+			)
+		)
 	)
 	(sheet

Commit message: Add files via upload
Parts:
- added J7: Conn_01x06_Socket, Connector_PinHeader_2.54mm:PinHeader_1x06_P2.54mm_Vertical, symbol Connector:Conn_01x06_Socket
Connections:
- net GND: now also J7.1 (Pin_1)
- net MCU_and_UI/ESP_RX: now also J7.4 (Pin_4)
- net MCU_and_UI/ESP_TX: now also J7.5 (Pin_5)
- net MCU_and_UI/ESP_boot: now also J7.6 (Pin_6)
- net MCU_and_UI/ESP_reset: now also J7.2 (Pin_2)
- net RX/RF: no longer C11.1, C12.1
- new net TX/RF_out: C11.1, C12.1
- no-connect marks 0 -> 1
Other:
- removed sheet channel_switching_and_filtering
- added sheet SWR_bridge (SWR_bridge.kicad_sch)
- sheet MCU_and_UI ports: added TX_Mod; removed TX_LO
- sheet TX ports: added RF_out, TX_Mod; removed RX_BFO

Commit message: Add files via upload
Other:
- moved on the sheet: C11, C12, J2, J7

Commit message: Add files via upload
Parts:
- added C1, C16, C2, C20, C21, C22, C33, C36, C7: 10n, Capacitor_SMD:C_0603_1608Metric_Pad1.08x0.95mm_HandSolder, symbol Device:C
- added C13, C14, C17, C24, C25, C31, C34, C35, C42, C52, C6, C63, C8: 100n, Capacitor_SMD:C_0603_1608Metric_Pad1.08x0.95mm_HandSolder, symbol Device:C
- added C15, C18, C32, C56, C57, C58, C59: 10u, Capacitor_SMD:C_1210_3225Metric_Pad1.33x2.70mm_HandSolder, symbol Device:C
- added C23: 10u, Capacitor_SMD:C_1210_3225Metric, symbol Device:C
- added C3, C4: 22p, Capacitor_SMD:C_0603_1608Metric_Pad1.08x0.95mm_HandSolder, symbol Device:C_Small
- added C37, C39, C53, C55: 150p, Capacitor_SMD:C_0603_1608Metric_Pad1.08x0.95mm_HandSolder, symbol Device:C
- added C41, C46: 470p, Capacitor_SMD:C_0603_1608Metric_Pad1.08x0.95mm_HandSolder, symbol Device:C
- added C49, C61: 1n, Capacitor_SMD:C_0603_1608Metric_Pad1.08x0.95mm_HandSolder, symbol Device:C
- added C5: 100n, Capacitor_SMD:C_0603_1608Metric_Pad1.08x0.95mm_HandSolder, symbol Device:C_Small
- added C54: 470u, Capacitor_THT:CP_Radial_D8.0mm_P3.80mm, symbol Device:C_Polarized
- added C9: 22p, Capacitor_SMD:C_0603_1608Metric_Pad1.08x0.95mm_HandSolder, symbol Device:C
- added D3, D4: D, Diode_SMD:D_PowerDI-123, symbol Device:D
- added D5: 1N4007, Diode_THT:D_A-405_P2.54mm_Vertical_AnodeUp, symbol Device:D
- added H1: Vin_+, TestPoint:TestPoint_THTPad_3.0x3.0mm_Drill1.5mm, symbol Mechanical:MountingHole_Pad
- added H2: Vin_-, TestPoint:TestPoint_THTPad_3.0x3.0mm_Drill1.5mm, symbol Mechanical:MountingHole_Pad
- added J3: PTT/Mic, Connector_Audio:Jack_3.5mm_CUI_SJ1-3525N_Horizontal, symbol summit_scourer:AudioJack2_Ground_Switch
- added J4: Headphone, Connector_Audio:Jack_3.5mm_CUI_SJ1-3525N_Horizontal, symbol summit_scourer:AudioJack2_Ground_Switch
- added J5: Internal_SPK, Connector_PinHeader_2.54mm:PinHeader_1x02_P2.54mm_Vertical, symbol Connector:Conn_01x02_Pin
- added J8: Conn_01x06_Socket, Connector_PinHeader_2.54mm:PinHeader_1x04_P2.54mm_Vertical, symbol Connector:Conn_01x04_Socket
- added L1: L, Inductor_THT:L_Toroid_Vertical_L10.0mm_W5.0mm_P5.08mm, symbol Device:L
- added L2, L5: L_Ferrite, Inductor_SMD:L_TDK_SLF6025, symbol Device:L_Ferrite
- added L3: 15T/T37-2, Inductor_THT:L_Toroid_Vertical_L10.0mm_W5.0mm_P5.08mm, symbol Device:L_Ferrite
- added L6: 10T/T37-2, Inductor_THT:L_Toroid_Vertical_L10.0mm_W5.0mm_P5.08mm, symbol Device:L_Ferrite
- added L8: L_Ferrite, Inductor_SMD:L_6.3x6.3_H3, symbol Device:L_Ferrite
- added MK1: Microphone, Connector_PinHeader_2.54mm:PinHeader_1x02_P2.54mm_Vertical, symbol Device:Microphone
- added Q1, Q3, Q4: BS170, Package_TO_SOT_THT:TO-92_Inline, symbol Transistor_FET:BS170
- added Q2: 2N7002H, Package_TO_SOT_SMD:SOT-23, symbol Transistor_FET:2N7002H
- added R1, R2, R25, R26, R27, R3, R32, R34, R4, R43, R50, R9: 0R, summit_scourer:R_0603_linked, symbol Device:R
- added R28, R29: 220R, Resistor_SMD:R_0603_1608Metric, symbol Device:R
- added R30, R31: 120k, Resistor_SMD:R_0603_1608Metric, symbol Device:R
- added R33, R40, R51, R54: 100k, Resistor_SMD:R_0603_1608Metric, symbol Device:R
- added R35, R42, R44, R45, R49, R52, R53, R6, R8: 10k, Resistor_SMD:R_0603_1608Metric, symbol Device:R
- added R41, R46, R47, R7: 1k, Resistor_SMD:R_0603_1608Metric, symbol Device:R
- added RV1: 10k, Connector_PinHeader_2.54mm:PinHeader_1x03_P2.54mm_Vertical, symbol Device:R_Potentiometer
- added SW7: Key, Connector_PinHeader_2.54mm:PinHeader_1x02_P2.54mm_Vertical, symbol Switch:SW_SPST
- added SW8: RotaryEncoder, summit_scourer:Rotary_encoder, symbol Device:RotaryEncoder_Switch
- added TP1: IO12, Connector_PinHeader_2.54mm:PinHeader_1x01_P2.54mm_Vertical, symbol Connector:TestPoint
- added U1: SI4732-A10-GS, Package_SO:SO-16_3.9x9.9mm_P1.27mm, symbol summit_scourer:SI4732-A10-GS
- added U3: Si5351A-B-GT, Package_SO:MSOP-10_3x3mm_P0.5mm, symbol Oscillator:Si5351A-B-GT
- added U4: ESP32-WROOM-32UE, RF_Module:ESP32-WROOM-32UE, symbol RF_Module:ESP32-WROOM-32UE
- added U5, U7: AZ1117-3.3, Package_TO_SOT_SMD:TO-252-2, symbol Regulator_Linear:AZ1117-3.3
- added U6: LM4808MX_NOPB, Package_SO:SO-8_3.9x4.9mm_P1.27mm, symbol summit_scourer:LM4808MX_NOPB
- added U8: 74AC00, Package_SO:SOIC-14_3.9x8.7mm_P1.27mm, symbol 74xx:74HC00
- added Y1: 32.768 KHz, Crystal:Crystal_SMD_3215-2Pin_3.2x1.5mm, symbol Device:Crystal_Small
- added Y3: 25MHz, Crystal:Crystal_SMD_3225-4Pin_3.2x2.5mm, symbol Device:Crystal_GND24_Small
- J7: value Conn_01x06_Socket -> Prog
Connections:
- net GND: now also C1.2, C13.2, C14.2, C16.2, C17.2, C20.2, C21.2, C23.2, C24.2, C25.2, C3.2, C31.2, C32.2, C33.2, C34.2, C35.2, C36.2, C37.2, C39.2, C4.2, C49.1, C52.2, C54.2, C56.2, C57.2, C58.2, C59.2, C6.2, C61.2, C63.2, C7.2, C9.2, D3.2 (A), D4.1 (K), H2.1, J3.S, J4.S, J5.2 (Pin_2), J8.4 (Pin_4), MK1.1 (-), Q1.3 (S), Q3.3 (S), Q4.3 (S), R28.2, R31.1, R33.2, R44.2, R52.2, R54.2, R8.2, SW7.2 (B), SW8.C, SW8.S2, U1.10 (SENB), U1.15 (GND), U1.7 (RFGND), U3.8 (GND), U4.1 (GND), U4.15 (GND), U4.38 (GND), U4.39 (GND), U5.1 (GND), U6.4 (GND), U6.5 (IN_B+), U6.6 (IN_B-), U7.1 (GND), U8.7 (GND), Y3.2, Y3.4
- net MCU_and_UI/ESP_RX renamed ESP_TX
- net ESP_TX: now also R3.2
- net MCU_and_UI/ESP_TX renamed ESP_reset
- net ESP_reset: now also C31.1, R40.2, U4.3 (EN)
- net MCU_and_UI/ESP_boot renamed ESP_RX
- net ESP_RX: now also R4.2
- net MCU_and_UI/ESP_reset renamed ESP_boot
- net ESP_boot: now also U4.25 (IO0)
- net TX/RF_out: no longer names the net of C11.1, C12.1
- net TX/RF_out: now also C53.2, C55.2, C61.1, L6.2
- new net: C32.1, C33.1, C35.1, L5.1, U4.2 (VDD)
- new net: C41.2, C46.2, L3.1
- new net: C49.2, C53.1, C55.1, L3.2, L6.1
- new net: R44.1, TP1.1, U4.14 (IO12)
- new net: R9.2, U3.1 (VDD)
- new net: J4.RN, J4.TN, J5.1 (Pin_1)
- new net: C18.2, RV1.1, U6.1 (OUT_A)
- new net: C2.2, C37.1, C39.1, C41.1, C46.1, L1.2, Q1.1 (D), Q3.1 (D), Q4.1 (D)
- new net: C22.1, U8.11, U8.3, U8.6
- new net: U8.1, U8.12, U8.4, U8.8
- new net: C14.1, C20.1, R34.2, U8.13, U8.14 (VCC), U8.2, U8.5, U8.9
- new net: C42.2, J3.R, R41.2
- new net: C21.1, R35.2, R53.1
- new net: U3.2 (XA), Y3.1
- new net: U3.3 (XB), Y3.3
- new net: R30.1, R31.2, U6.3 (IN_A+)
- new net: R4.1, U4.34 (RXD0/IO3)
- new net: C4.1, U1.2 (GPO3/DCLK), Y1.1
- new net: C3.1, U1.13 (RCLK), Y1.2
- new net: R1.2, U3.4 (SCL)
- new net: C5.1, D3.1 (K), D4.2 (A), Q2.3 (D)
- new net: C5.2, U1.8 (AMI)
- new net: R29.1, U1.4 (GPO1)
- new net: C13.1, C16.1, L2.1, R29.2, U1.14 (VDD)
- new net: C22.2, Q1.2 (G), Q3.2 (G), Q4.2 (G), R53.2, R54.1
- new net: RV1.2, U6.2 (IN_A-)
- new net: R7.2, RV1.3
- new net: D5.1 (K), L8.1
- new net: C2.1, Q2.2 (S)
- new net: R25.1, U1.12 (SDIO)
- new net: R26.1, U1.11 (SCLK)
- new net: C8.1, C9.1, R33.1, U8.10
- new net: R43.1, U4.24 (IO2)
- new net: R3.1, U4.35 (TXD0/IO1)
- new net: R28.1, U1.3 (GPO2/INTB)
- new net: C15.1, U1.16 (ROUT/DOUT)
- new net: C15.2, R7.1
- new net: R27.1, U1.9 (~{RST})
- new net: C8.2, U3.10 (CLK0)
- new net: R2.2, U3.5 (SDA)
- new net: R32.2, U3.7 (VDDO)
- new net +3V3: C58.1, C6.1, C63.1, C7.1, J8.3 (Pin_3), L5.2, R32.1, R34.1, R40.1, R41.1, R42.1, R45.2, R46.1, R47.1, R50.1, R6.1, R9.1, U5.2 (VO)
- new net +3V3_RX: C17.1, C59.1, L2.2, R30.2, R50.2, U6.8 (VDD), U7.2 (VO)
- new net Encoder.A: SW8.A, U4.36 (IO22)
- new net Encoder.B: SW8.B, U4.37 (IO23)
- new net Encoder.btn: C25.1, R6.2, SW8.S1, U4.12 (IO27)
- new net I2C_SCL: J8.2 (Pin_2), R1.1, R26.2, R46.2, U4.29 (IO5)
- new net I2C_SDIO: J8.1 (Pin_1), R2.1, R25.2, R47.2, U4.26 (IO4)
- new net PTT_key: C34.1, J3.T, R42.2, U4.7 (IO35)
- new net RX_ant_en: C1.1, Q2.1 (G), R43.2
- new net TX_Mod: R35.1, U4.10 (IO25)
- new net VBUS: C23.1, C24.1, C52.1, D5.2 (A), H1.1, L1.1
- new net VBUS_filtered: C54.1, C56.1, C57.1, L8.2, R51.1, U5.3 (VI), U7.3 (VI)
- new net V_sense: R51.2, R52.1, U4.13 (IO14)
- new net audio_out_right: C18.1, J4.R, J4.T, R49.2
- new net mic_in: C36.1, C42.1, R45.1, R8.1, U4.6 (IO34)
- new net onboard_key: J3.TN, SW7.1 (A)
- new net onboard_mic: J3.RN, MK1.2 (+)
- new net side_tone: R49.1, U4.11 (IO26)
- new net ~{SI_RST}: R27.2, U4.16 (IO13)
- no-connect marks 1 -> 6
Other:
- removed sheet MCU_and_UI
- removed sheet PSU
- removed sheet RX
- removed sheet SWR_bridge
- removed sheet TX
- note added: "40m"
- note added: "ESP32 Input only pins: Name Num Sensor_VP 4 Sensor_VN 5 IO34 6 IO35 7 DAC pins: Name Num DAC name IO24 10 DAC_1 IO26 11 DAC_2"
- moved on the sheet: C11, C12, J2, J7

Commit message: Add files via upload
Connections:
- net Encoder.A: now also U4.31 (IO19); no longer U4.36 (IO22)
- net I2C_SCL: now also U4.36 (IO22); no longer U4.29 (IO5)
- net I2C_SDIO: now also U4.33 (IO21); no longer U4.26 (IO4)
Other:
- moved on the sheet: C18, C42, R51, R52, R8
