File: summit_scourer.kicad_sch (KiCad schematic)
At the start: 115 parts, among them J2 Conn_Coaxial, J3 PTT/Mic, J4 Headphone, J5 Internal_SPK, J7 Prog, J8 Conn_01x06_Socket, Q1 BS170, Q2 2N7002H, Q3 BS170, Q4 BS170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

Commit message: Add files via upload
Parts:
- added H3: ANT, TestPoint:TestPoint_THTPad_3.0x3.0mm_Drill1.5mm, symbol Mechanical:MountingHole_Pad
- added H4: GND, TestPoint:TestPoint_THTPad_3.0x3.0mm_Drill1.5mm, symbol Mechanical:MountingHole_Pad
Connections:
- net GND: now also H4.1
- net at C11.2, C12.2, J2.1 (In): now also H3.1
Other:
- moved on the sheet: C11, C12, J2
