File: summit_scourer.kicad_pcb (KiCad board)
At the start: 4 copper layers, 78 x 47 mm, 115 parts, among them J2 Conn_Coaxial, J3 PTT/Mic, J4 Headphone, J5 Internal_SPK, J7 Prog, J8 Conn_01x06_Socket, Q1 BS170, Q2 2N7002H, Q3 BS170, Q4 BS170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

Commit message: Add files via upload
Parts:
- added H3: ANT, TestPoint:TestPoint_THTPad_3.0x3.0mm_Drill1.5mm, F.Cu at (181.8, 111.5)
- added H4: GND, TestPoint:TestPoint_THTPad_3.0x3.0mm_Drill1.5mm, F.Cu at (181.8, 116.5)
- moved C11 8.31 mm to (184.9, 96.4)
- moved C12 8.31 mm to (183.3, 96.4)
- moved C49 8.04 mm to (177.7, 89.5), turned to 0 degrees
- moved J2 6.99 mm to (181.8, 103.8)
- moved C53 6.65 mm to (181.6, 94.6)
- moved C55 6.65 mm to (179.6, 94.6)
- moved C61 6.65 mm to (177.8, 97.2)
- moved L6 6.65 mm to (180.7, 92.0)
- moved L3 4.81 mm to (180.7, 84.4)
- moved C37 0.83 mm to (183.9, 87.0)
- moved C39 0.83 mm to (185.5, 87.0)
- moved C41 0.83 mm to (181.3, 86.1)
- moved C46 0.83 mm to (181.3, 87.6)
Routing:
- net Net-(J2-In): track 7.70 -> 16.5 mm
- net Net-(C11-Pad1): track 9.97 -> 8.86 mm
- net Net-(C41-Pad2): track 4.13 -> 3.30 mm
- net Net-(Q1-D): track 47.1 -> 47.7 mm
- net GND: vias 182 -> 179

Commit message: Add files via upload
Parts:
- moved R49 3.00 mm to (122.8, 104.0), turned to 90 degrees
- moved J7 2.80 mm to (108.7, 119.1)
- moved R41 2.15 mm to (112.7, 87.8)
- moved J3 2.03 mm to (110.8, 95.2)
- moved J4 2.03 mm to (110.8, 82.2)
- moved C34 2.00 mm to (112.6, 100.8)
- moved C42 2.00 mm to (113.3, 91.2)
- moved R42 2.00 mm to (111.2, 98.0)
- moved R45 2.00 mm to (111.1, 92.2)
- moved R8 2.00 mm to (113.3, 94.5)
- moved J5 1.48 mm to (121.1, 79.7)
- moved MK1 1.48 mm to (121.1, 90.0)
- moved SW7 1.48 mm to (121.1, 98.0)
- moved RV1 1.21 mm to (128.7, 78.5)
- moved U4 0.45 mm to (136.7, 109.4)
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Routing:
- net /side_tone: track 1.78 -> 5.31 mm
- net /I2C_SDIO: track 44.2 -> 41.2 mm
- net /ESP_boot: track 46.8 -> 49.7 mm
- net /ESP_reset: track 22.9 -> 25.2 mm
- net /ESP_TX: track 29.7 -> 31.8 mm
- net Net-(U6-OUT_A): track 18.6 -> 17.0 mm
- net /ESP_RX: track 25.2 -> 26.6 mm
- net /PTT_key: track 23.5 -> 24.8 mm
- net Net-(R7-Pad2): track 45.0 -> 43.8 mm
- net Net-(U6-IN_A-): track 14.4 -> 13.4 mm
- net /I2C_SCL: track 42.7 -> 41.7 mm
- net /onboard_mic: track 4.85 -> 5.40 mm
- net /onboard_key: track 4.85 -> 5.40 mm
- net GND: track 15.3 -> 15.6 mm, vias 179 -> 177
- net /audio_out_right: track 39.3 -> 39.5 mm, vias 2 -> 0
Other:
- board size 78 x 47 mm -> 80 x 47.5 mm
- board text added: "AF Gain"
